Commit message: Stable gazebo wam_powerbot.urdf file: changes: - reduced the height of the asus camera - pushed the wheels towards the front of the chassis for stability.

File: champ_description/urdf/asus/asus.xacro (robot description, xacro)
@@ -29,5 +29,5 @@
           <origin xyz="0 0 0" rpy="0 0 0" />
           <geometry>
-            <box size="0.06 0.25 0.05"/>   <!--box size="0.035 0.185 0.025"/-->
+           <mesh filename="${asus_mesh_directory}/asus_camera_simple.dae"/>  <!--box size="0.035 0.185 0.025"/-->
           </geometry>
         </collision>

File: champ_description/urdf/asus/asus_cal.xacro (robot description, xacro)
@@ -3,5 +3,5 @@
 <xacro:property name="asus_x" value="0.451798"/>
 <xacro:property name="asus_y" value="0.0081349"/><!-- 0.0581349 -->
-<xacro:property name="asus_z" value="0.561428"/>
+<xacro:property name="asus_z" value="0.461428"/>
 <xacro:property name="asus_roll" value="0.0202643"/><!-- -0.0172643 -->
 <xacro:property name="asus_pitch" value="0.415979"/><!-- 0.425979 -->

File: champ_description/urdf/powerbot/powerbot.urdf (robot description, URDF)
Before this commit: robot powerbot, 15 links, 14 joints
Joints:
- joint left_hub_joint: origin xyz=0.034 0.35 -0.0835 rpy=0 0 0 -> xyz=0.084 0.35 -0.0835 rpy=0 0 0
- joint right_hub_joint: origin xyz=0.034 -0.35 -0.0835 rpy=0 0 0 -> xyz=0.084 -0.35 -0.0835 rpy=0 0 0

File: champ_description/urdf/powerbot/powerbot.xacro (robot description, xacro)
@@ -5,4 +5,12 @@
 	xmlns:interface="http://playerstage.sourceforge.net/gazebo/xmlschema/#interface"
 	xmlns:xacro="http://ros.org/wiki/xacro">
+ <!-- robot name -->
+  <xacro:macro name="powerbot" params="prefix parent_link xyz rpy">
+    <joint name ="${prefix}/world_joint" type="planar">
+      <parent link="${parent_link}"/>
+      <child link="base_center"/>
+      <origin xyz="${xyz}" rpy="${rpy}"/>
+    </joint>
+  </xacro:macro>
   <!-- Include powerbot wheels -->
   <xacro:include filename="$(find champ_description)/urdf/powerbot/powerbot_wheel.xacro"/>
@@ -201,5 +209,5 @@
 		<anchor xyz="0 0 0"/>
     <limit effort="100" velocity="100" k_velocity="0" />
-    <joint_properties damping="0.0" friction="0.0" />
+    <joint_properties damping="7.0" friction="0.0" />
 	  <parent link="right_swivel"/>
 		<child link="right_swivel_hubcap"/>
@@ -335,5 +343,5 @@
 		<anchor xyz="0 0 0"/>
     <limit effort="100" velocity="100" k_velocity="0" />
-    <joint_properties damping="0.0" friction="0.0" />
+    <joint_properties damping="7.0" friction="0.0" />
 	  <parent link="left_swivel"/>
 		<child link="left_swivel_hubcap"/>
@@ -395,5 +403,5 @@
 	</link>
 	<joint name="left_hub_joint" type="fixed">
-		<origin xyz="0.034 0.35 -0.0835" rpy="0 0 0"/>
+		<origin xyz="0.084 0.35 -0.0835" rpy="0 0 0"/>
 	        <!--<anchor xyz="0 0 0"/>
 	        <limit effort="100" velocity="100" />
@@ -459,5 +467,5 @@
 	</link>
 	<joint name="right_hub_joint" type="fixed">
-		<origin xyz="0.034 -0.35 -0.0835" rpy="0 0 0"/>
+		<origin xyz="0.084 -0.35 -0.0835" rpy="0 0 0"/>
 	        <!--<anchor xyz="0 0 0"/>
 	        <limit effort="100" velocity="100" />

File: champ_description/urdf/wam_powerbot.urdf (robot description, URDF)
Before this commit: robot wam_powerbot, 44 links, 43 joints
Links:
- removed link back_sonar
- removed link center_hubcap
- removed link center_hubcap2
- removed link center_wheel
- removed link center_wheel2
- removed link front_sonar
- removed link left_hub
- removed link left_wheel_joint
- removed link right_hub
- removed link right_wheel_joint
- removed link swivel
- removed link swivel2
- added link left_hubcap, mass 0.08; collision mesh filename=package://champ_description/meshes/p3dx_meshes/hubcap.stl; visual mesh filename=package://champ_description/meshes/p3dx_meshes/hubcap.stl
- added link left_swivel, mass 0.1; collision mesh filename=package://champ_description/meshes/p3dx_meshes/swivel.stl; visual mesh filename=package://champ_description/meshes/p3dx_meshes/swivel.stl
- added link left_swivel_hubcap, mass 0.01; collision mesh filename=package://champ_description/meshes/p3dx_meshes/center_hubca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; visual mesh filename=package://champ_description/meshes/p3dx_meshes/center_hubca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
- added link left_swivel_support, mass 0.1; collision mesh filename=package://champ_description/meshes/p3dx_meshes/swivel_suppo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; visual mesh filename=package://champ_description/meshes/p3dx_meshes/swivel_suppo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
- added link left_swivel_wheel, mass 0.1; collision cylinder length=0.0422 radius=0.0669; visual mesh filename=package://champ_description/meshes/p3dx_meshes/center_wheel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
- added link left_wheel, mass 1.25; collision cylinder length=0.065 radius=0.1315; visual mesh filename=package://champ_description/meshes/p3dx_meshes/wheel.stl
- added link right_hubcap, mass 0.08; collision mesh filename=package://champ_description/meshes/p3dx_meshes/hubcap.stl; visual mesh filename=package://champ_description/meshes/p3dx_meshes/hubcap.stl
- added link right_swivel, mass 0.1; collision mesh filename=package://champ_description/meshes/p3dx_meshes/swivel.stl; visual mesh filename=package://champ_description/meshes/p3dx_meshes/swivel.stl
- added link right_swivel_hubcap, mass 0.01; collision mesh filename=package://champ_description/meshes/p3dx_meshes/center_hubca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; visual mesh filename=package://champ_description/meshes/p3dx_meshes/center_hubca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
- added link right_swivel_support, mass 0.1; collision mesh filename=package://champ_description/meshes/p3dx_meshes/swivel_suppo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; visual mesh filename=package://champ_description/meshes/p3dx_meshes/swivel_suppo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
- added link right_swivel_wheel, mass 0.1; collision cylinder length=0.0422 radius=0.0669; visual mesh filename=package://champ_description/meshes/p3dx_meshes/center_wheel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
- added link right_wheel, mass 1.25; collision cylinder length=0.065 radius=0.1315; visual mesh filename=package://champ_description/meshes/p3dx_meshes/wheel.stl
- link kinect_link: geometry collision mesh filename=package://champ_description/meshes/asus_camera/asus_camera_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; visual mesh filename=package://champ_description/meshes/asus_camera/asus_camera_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
- link top_plate: geometry collision mesh filename=package://champ_description/meshes/p3dx_meshes/top.stl; visual mesh filename=package://champ_description/meshes/p3dx_meshes/top.stl
Joints:
- removed joint base_back_joint
- removed joint base_front_joint
- removed joint base_swivel_joint
- removed joint base_swivel_joint2
- removed joint center_wheel_joint
- removed joint center_wheel_joint2
- removed joint swivel_hubcap_joint
- removed joint swivel_hubcap_joint2
- added joint left_base_swivel_joint: type fixed, parent left_swivel_support, child left_swivel, origin xyz=0 0 -0.04855 rpy=0 0 0
- added joint left_base_swivel_support_joint: type fixed, parent base_center, child left_swivel_support, origin xyz=-0.215 0.2 -0.091 rpy=0 0 0
- added joint left_swivel_hubcap_joint: type continuous, parent left_swivel, child left_swivel_hubcap, origin xyz=-0.036 0 -0.029 rpy=0 0 0, axis 0 1 0, limit effort=100 velocity=100
- added joint left_swivel_wheel_hubcap_joint: type fixed, parent left_swivel_hubcap, child left_swivel_wheel, origin xyz=0 0 0 rpy=0 0 0
- added joint right_base_swivel_joint: type fixed, parent right_swivel_support, child right_swivel, origin xyz=0 0 -0.04855 rpy=0 0 0
- added joint right_base_swivel_support_joint: type fixed, parent base_center, child right_swivel_support, origin xyz=-0.215 -0.2 -0.091 rpy=0 0 0
- added joint right_swivel_hubcap_joint: type continuous, parent right_swivel, child right_swivel_hubcap, origin xyz=-0.036 0 -0.029 rpy=0 0 0, axis 0 1 0, limit effort=100 velocity=100
- added joint right_swivel_wheel_hubcap_joint: type fixed, parent right_swivel_hubcap, child right_swivel_wheel, origin xyz=0 0 0 rpy=0 0 0
- joint base_top_joint: origin xyz=-0.045 0 0.3085 rpy=0 0 0 -> xyz=-0.045 0 0.277 rpy=0 0 0
- joint kinect_joint: origin xyz=0.451798 0.0081349 0.561428 rpy=0.0202643 0.415979 0.0134257 -> xyz=0.451798 0.0081349 0.461428 rpy=0.0202643 0.415979 0.0134257
- joint left_hub_joint: child left_hub -> left_hubcap; origin xyz=0.1 0.30 0.0235 rpy=0 0 0 -> xyz=0.034 0.35 -0.0835 rpy=0 0 0
- joint left_wheel_joint: child left_wheel_joint -> left_wheel; parent left_hub -> left_hubcap
- joint right_hub_joint: child right_hub -> right_hubcap; origin xyz=0.1 -0.30 0.0235 rpy=0 0 0 -> xyz=0.034 -0.35 -0.0835 rpy=0 0 0
- joint right_wheel_joint: child right_wheel_joint -> right_wheel; parent right_hub -> right_hubcap
