Commit message: Added kinect from turtlebot_description and position it at origin from asus_cal Issues: 	- Missing differential drive controller 	- Joint PID params untuned

File: champ_description/urdf/asus/asus_cal.xacro (robot description, xacro)
@@ -1,7 +1,7 @@
 <?xml version="1.0"?>
 <robot xmlns:xacro="http://ros.org/wiki/xacro">
-<xacro:property name="asus_x" value="0.451798"/>
+<xacro:property name="asus_x" value="0.351798"/>
 <xacro:property name="asus_y" value="0.0081349"/><!-- 0.0581349 -->
-<xacro:property name="asus_z" value="0.461428"/>
+<xacro:property name="asus_z" value="0.16"/>
 <xacro:property name="asus_roll" value="0.0202643"/><!-- -0.0172643 -->
 <xacro:property name="asus_pitch" value="0.415979"/><!-- 0.425979 -->

File: champ_description/urdf/wam_powerbot.xacro (robot description, xacro)
@@ -7,7 +7,17 @@
   <!-- Includea all the WAM stuff -->
   <xacro:include filename="$(find champ_description)/urdf/wam/wam_top.urdf.xacro"/>
+<link name="cam"/>
   <!-- Include powerbot -->
-  <xacro:include filename="$(find champ_description)/urdf/powerbot/powerbot.xacro"/>
-<!-- Kinect stuff -->
+ <xacro:include filename="$(find champ_description)/urdf/powerbot/powerbot.xacro"/>
+<!-- Load kinect from turtlebot_description and position it at origin from asus_cal -->
+<xacro:include filename="$(find champ_description)/urdf/asus/asus_cal.xacro"/>
+<xacro:include filename="$(find turtlebot_description)/urdf/sensors/asus_xtion_pro.urdf.xacro"/>
+<xacro:sensor_asus_xtion_pro parent="cam"/>
+<joint name="cam_joint" type="fixed">
+	<origin xyz="${asus_x} ${asus_y} ${asus_z}" rpy="${asus_roll} ${asus_pitch} ${asus_yaw}"/>
+	<parent link="base_center"/>
+	<child link="cam"/>
+</joint>
+<!-- Kinect stuff
   <xacro:include filename="$(find champ_description)/urdf/asus/asus.xacro"/>
   <xacro:include filename="$(find champ_description)/urdf/asus/asus_cal.xacro"/>
@@ -15,4 +25,5 @@
        <origin xyz="${asus_x} ${asus_y} ${asus_z}" rpy="${asus_roll} ${asus_pitch} ${asus_yaw}"/>
   </xacro:asus_camera_model>
+  -->
 <!-- Root link is in the world frame-->
 <link name="world"/>
