Commit message: Added joint efort controllers controllers for all wam joints. Issues:  - finger links jump around when controller is started  - swivel_to_base_center joints still "fixed" instead of continuous  - Champ robot slides away from origin in gazebo. 	- Explore friction tag in powerbot.xacro file  - No controllers for base wheels have been implemented yet. 	-  look at differential drive controller.

File: champ_description/urdf/wam/hand.urdf.xacro (robot description, xacro)
@@ -132,4 +132,9 @@
       <limit effort="5" lower="0" upper="${PI}" velocity="5.0"/>
       <dynamics damping="${0.1*b}" friction="0"/>
+<!--
+	<xacro:if value= "${prefix=='wam/bhand/finger_2'}">
+	  <mimic joint="wam/bhand/finger_1/prox_joint" multiplier="-1.0" offset="0.0" />
+	</xacro:if>
+-->
     </joint>
     <gazebo reference="${prefix}/prox_joint">

File: champ_description/urdf/wam_powerbot.urdf (robot description, URDF)
Before this commit: robot wam_powerbot, 44 links, 43 joints
Joints:
- joint left_hub_joint: origin xyz=0.034 0.35 -0.0835 rpy=0 0 0 -> xyz=0.084 0.35 -0.0835 rpy=0 0 0
- joint right_hub_joint: origin xyz=0.034 -0.35 -0.0835 rpy=0 0 0 -> xyz=0.084 -0.35 -0.0835 rpy=0 0 0

File: champ_description/urdf/wam_powerbot.xacro (robot description, xacro)
@@ -19,7 +19,193 @@
 <!-- ArmStuff -->
 <!-- BHand -->
-<xacro:bhand prefix="wam/bhand" parent_link="wam/wrist_palm_link" xyz="0 0 0.06" rpy="0 0 0"/>
+<xacro:bhand prefix="wam/bhand" parent_link="wam/wrist_palm_link" xyz="0 0 0.1" rpy="0 0 0"/>
 <!-- 7-DOF Wam on top of top plate-->
 <xacro:wam_7dof prefix="wam" parent_link="arm_plate" xyz="0.22 0.0 0.05" rpy="0 0 0" />
 <xacro:powerbot prefix="powerbot" parent_link="world" xyz="0.0 0.0 0.0" rpy="0 0 0" />
+<!--Joint Controllers
+- ARM
+      - wam/base_yaw_joint
+      - wam/shoulder_pitch_joint
+      - wam/shoulder_yaw_joint
+      - wam/elbow_pitch_joint
+      - wam/wrist_yaw_joint
+      - wam/wrist_pitch_joint
+      - wam/palm_yaw_joint
+- HAND
+      - wam/bhand/finger_1/med_joint
+      - wam/bhand/finger_1/dist_joint
+      - wam/bhand/finger_2/med_joint
+      - wam/bhand/finger_2/dist_joint
+      - wam/bhand/finger_3/dist_joint
+-->
+<!-- wam/base_yaw_joint -->
+  <transmission name="w1">
+    <type>transmission_interface/SimpleTransmission</type>
+    <joint name="wam/base_yaw_joint">
+      <hardwareInterface>hardware_interface/EffortJointInterface</hardwareInterface>
+    </joint>
+    <actuator name="motor1">
+      <hardwareInterface>hardware_interface/EffortJointInterface</hardwareInterface>
+      <mechanicalReduction>1</mechanicalReduction>
+    </actuator>
+  </transmission>
+<!-- wam/shoulder_pitch_joint -->
+  <transmission name="w2">
+    <type>transmission_interface/SimpleTransmission</type>
+    <joint name="wam/shoulder_pitch_joint">
+      <hardwareInterface>hardware_interface/EffortJointInterface</hardwareInterface>
+    </joint>
+    <actuator name="motor2">
+      <hardwareInterface>hardware_interface/EffortJointInterface</hardwareInterface>
+      <mechanicalReduction>1</mechanicalReduction>
+    </actuator>
+  </transmission>
+<!-- wam/shoulder_yaw_joint -->
+  <transmission name="w3">
+    <type>transmission_interface/SimpleTransmission</type>
+    <joint name="wam/shoulder_yaw_joint">
+      <hardwareInterface>hardware_interface/EffortJointInterface</hardwareInterface>
+    </joint>
+    <actuator name="motor3">
+      <hardwareInterface>hardware_interface/EffortJointInterface</hardwareInterface>
+      <mechanicalReduction>1</mechanicalReduction>
+    </actuator>
+  </transmission>
+<!-- wam/elbow_pitch_joint -->
+  <transmission name="w4">
+    <type>transmission_interface/SimpleTransmission</type>
+    <joint name="wam/elbow_pitch_joint">
+      <hardwareInterface>hardware_interface/EffortJointInterface</hardwareInterface>
+    </joint>
+    <actuator name="motor4">
+      <hardwareInterface>hardware_interface/EffortJointInterface</hardwareInterface>
+      <mechanicalReduction>1</mechanicalReduction>
+    </actuator>
+  </transmission>
+<!-- wam/wrist_yaw_joint -->
+  <transmission name="w5">
+    <type>transmission_interface/SimpleTransmission</type>
+    <joint name="wam/wrist_yaw_joint">
+      <hardwareInterface>hardware_interface/EffortJointInterface</hardwareInterface>
+    </joint>
+    <actuator name="motor5">
+      <hardwareInterface>hardware_interface/EffortJointInterface</hardwareInterface>
+      <mechanicalReduction>1</mechanicalReduction>
+    </actuator>
+  </transmission>
+<!-- wam/wrist_pitch_joint -->
+  <transmission name="w6">
+    <type>transmission_interface/SimpleTransmission</type>
+    <joint name="wam/wrist_pitch_joint">
+      <hardwareInterface>hardware_interface/EffortJointInterface</hardwareInterface>
+    </joint>
+    <actuator name="motor6">
+      <hardwareInterface>hardware_interface/EffortJointInterface</hardwareInterface>
+      <mechanicalReduction>1</mechanicalReduction>
+    </actuator>
+  </transmission>
+<!-- wam/palm_yaw_joint -->
+  <transmission name="w7">
+    <type>transmission_interface/SimpleTransmission</type>
+    <joint name="wam/palm_yaw_joint">
+      <hardwareInterface>hardware_interface/EffortJointInterface</hardwareInterface>
+    </joint>
+    <actuator name="motor7">
+      <hardwareInterface>hardware_interface/EffortJointInterface</hardwareInterface>
+      <mechanicalReduction>1</mechanicalReduction>
+    </actuator>
+  </transmission>
+<!-- wam/bhand/finger_1/prox_joint -->
+  <transmission name="f1_prox">
+    <type>transmission_interface/SimpleTransmission</type>
+    <joint name="wam/bhand/finger_1/prox_joint">
+      <hardwareInterface>hardware_interface/EffortJointInterface</hardwareInterface>
+    </joint>
+    <actuator name="motor8_1">
+      <hardwareInterface>hardware_interface/EffortJointInterface</hardwareInterface>
+      <mechanicalReduction>1</mechanicalReduction>
+    </actuator>
+  </transmission>
+<!-- wam/bhand/finger_1/med_joint -->
+  <transmission name="f1_med">
+    <type>transmission_interface/SimpleTransmission</type>
+    <joint name="wam/bhand/finger_1/med_joint">
+      <hardwareInterface>hardware_interface/EffortJointInterface</hardwareInterface>
+    </joint>
+    <actuator name="motor8_2">
+      <hardwareInterface>hardware_interface/EffortJointInterface</hardwareInterface>
+      <mechanicalReduction>1</mechanicalReduction>
+    </actuator>
+  </transmission>
+<!-- wam/bhand/finger_1/dist_joint -->
+  <transmission name="f1_dist">
+    <type>transmission_interface/SimpleTransmission</type>
+    <joint name="wam/bhand/finger_1/dist_joint">
+      <hardwareInterface>hardware_interface/EffortJointInterface</hardwareInterface>
+    </joint>
+    <actuator name="motor8_3">
+      <hardwareInterface>hardware_interface/EffortJointInterface</hardwareInterface>
+      <mechanicalReduction>1</mechanicalReduction>
+    </actuator>
+  </transmission>
+<!-- wam/bhand/finger_2/prox_joint -->
+  <transmission name="f2_prox">
+    <type>transmission_interface/SimpleTransmission</type>
+    <joint name="wam/bhand/finger_2/prox_joint">
+      <hardwareInterface>hardware_interface/EffortJointInterface</hardwareInterface>
+    </joint>
+    <actuator name="motor9_1">
+      <hardwareInterface>hardware_interface/EffortJointInterface</hardwareInterface>
+      <mechanicalReduction>1</mechanicalReduction>
+    </actuator>
+  </transmission>
+<!-- wam/bhand/finger_2/med_joint -->
+  <transmission name="f2_med">
+    <type>transmission_interface/SimpleTransmission</type>
+    <joint name="wam/bhand/finger_2/med_joint">
+      <hardwareInterface>hardware_interface/EffortJointInterface</hardwareInterface>
+    </joint>
+    <actuator name="motor9_2">
+      <hardwareInterface>hardware_interface/EffortJointInterface</hardwareInterface>
+      <mechanicalReduction>1</mechanicalReduction>
+    </actuator>
+  </transmission>
+<!-- wam/bhand/finger_2/dist_joint -->
+  <transmission name="f2_dist">
+    <type>transmission_interface/SimpleTransmission</type>
+    <joint name="wam/bhand/finger_2/dist_joint">
+      <hardwareInterface>hardware_interface/EffortJointInterface</hardwareInterface>
+    </joint>
+    <actuator name="motor9_3">
+      <hardwareInterface>hardware_interface/EffortJointInterface</hardwareInterface>
+      <mechanicalReduction>1</mechanicalReduction>
+    </actuator>
+  </transmission>
+<!-- wam/bhand/finger_3/med_joint -->
+  <transmission name="f3_med">
+    <type>transmission_interface/SimpleTransmission</type>
+    <joint name="wam/bhand/finger_3/med_joint">
+      <hardwareInterface>hardware_interface/EffortJointInterface</hardwareInterface>
+    </joint>
+    <actuator name="motor10_1">
+      <hardwareInterface>hardware_interface/EffortJointInterface</hardwareInterface>
+      <mechanicalReduction>1</mechanicalReduction>
+    </actuator>
+  </transmission>
+<!-- wam/bhand/finger_3/dist_joint -->
+  <transmission name="f3_dist">
+    <type>transmission_interface/SimpleTransmission</type>
+    <joint name="wam/bhand/finger_3/dist_joint">
+      <hardwareInterface>hardware_interface/EffortJointInterface</hardwareInterface>
+    </joint>
+    <actuator name="motor10_2">
+      <hardwareInterface>hardware_interface/EffortJointInterface</hardwareInterface>
+      <mechanicalReduction>1</mechanicalReduction>
+    </actuator>
+  </transmission>
+<gazebo>
+  <plugin name="gazebo_ros_control" filename="libgazebo_ros_control.so">
+    <robotNamespace>/wam_powerbot</robotNamespace>
+  </plugin>
+</gazebo>
 </robot>
