Commit message: - Added effort controllers for WAM gazebo model: 	- Created separate launch files for effort and position controllers. - Started moduralising WAM gazebo model: 	- Created separate launch and xacro files for WAM with Barrett hand and Ball (no hand).
TODO:
	- Move WAM joint jontroller definitions from wam_powerbot.xacro to wam7_bball.urdf.xacro
	  and wam7_bhand.urdf.xacro.
	- Place unrelated WAM xacro files in a subfolder.
ISSUES:
	- WAM collision meshes have holes.
        - WAM joint PID parameters still untuned.
        - Rviz does not visualise joint states topic (Mismatching msg types?).
	deleted:    CMakeLists.txt
	modified:   champ_description/launch/champ_world.launch
	modified:   champ_description/launch/empty.world
	renamed:    champ_description/gazebo/powerbot-empty-world.launch -> champ_description/launch/powerbot.launch
	renamed:    champ_description/gazebo/wam-empty-world.launch -> champ_description/launch/wam_bball.launch
	new file:   champ_description/launch/wam_bhand.launch
	new file:   champ_description/urdf/wam/wam7_bball.urdf.xacro
	modified:   champ_description/urdf/wam/wam7_bhand.urdf.xacro
	new file:   champ_description/urdf/wam/wam_bball.urdf
	renamed:    champ_description/urdf/wam/wam7_bhand.urdf -> champ_description/urdf/wam/wam_bhand.urdf
	new file:   champ_description/urdf/wam_ball.xacro
	new file:   champ_description/urdf/wam_ball_powerbot.xacro
	new file:   champ_description/urdf/wam_bhand_powerbot.xacro
	modified:   champ_description/urdf/wam_powerbot.urdf
	modified:   champ_description/urdf/wam_powerbot.xacro
	new file:   wam_control/config/wam_control_effort.yaml
	renamed:    wam_control/config/wam_control.yaml -> wam_control/config/wam_control_position.yaml
	new file:   wam_control/launch/wam_control_effort.launch
	renamed:    wam_control/launch/wam_control.launch -> wam_control/launch/wam_control_position.launch

File: champ_description/urdf/wam/wam7_bball.urdf.xacro (robot description, xacro)
@@ -8,6 +8,5 @@
   <!-- 7-DOF Wam -->
   <xacro:wam_7dof prefix="wam" parent_link="world" xyz="0.0 0.0 0.5" rpy="0 0 0" />
-  <!-- BHand -->
-  <xacro:bhand prefix="wam/bhand" parent_link="wam/wrist_palm_link" xyz="0 0 0.06" rpy="0 0 1.57079"/>
-  <!-- WAM joint Controllers -->
+  <!-- BBall -->
+  <xacro:bball prefix="wam/bball" parent_link="wam/wrist_palm_link" xyz="0 0 0.06" rpy="0 0 1.57079"/>
 </robot>

File: champ_description/urdf/wam/wam_bball.urdf (robot description, URDF)
Before this commit: robot wam, 24 links, 23 joints
Links:
- removed link wam/bhand/bhand_grasp_link
- removed link wam/bhand/bhand_palm_link
- removed link wam/bhand/bhand_palm_surface_link
- removed link wam/bhand/finger_1/dist_link
- removed link wam/bhand/finger_1/med_link
- removed link wam/bhand/finger_1/prox_link
- removed link wam/bhand/finger_1/tip_link
- removed link wam/bhand/finger_2/dist_link
- removed link wam/bhand/finger_2/med_link
- removed link wam/bhand/finger_2/prox_link
- removed link wam/bhand/finger_2/tip_link
- removed link wam/bhand/finger_3/dist_link
- removed link wam/bhand/finger_3/med_link
- removed link wam/bhand/finger_3/tip_link
- added link wam/bball/bball_base_link, mass 0.5986; collision cylinder length=0.01 radius=0.0415; collision cylinder length=0.065 radius=0.006
- added link wam/bball/bball_center_link, mass 0.00001
Joints:
- removed joint wam/bhand/bhand_base_joint
- removed joint wam/bhand/bhand_grasp_joint
- removed joint wam/bhand/bhand_palm_surface_joint
- removed joint wam/bhand/finger_1/dist_joint
- removed joint wam/bhand/finger_1/med_joint
- removed joint wam/bhand/finger_1/prox_joint
- removed joint wam/bhand/finger_1/tip_joint
- removed joint wam/bhand/finger_2/dist_joint
- removed joint wam/bhand/finger_2/med_joint
- removed joint wam/bhand/finger_2/prox_joint
- removed joint wam/bhand/finger_2/tip_joint
- removed joint wam/bhand/finger_3/dist_joint
- removed joint wam/bhand/finger_3/med_joint
- removed joint wam/bhand/finger_3/tip_joint
- added joint wam/bball/bball_base_joint: type fixed, parent wam/wrist_palm_link, child wam/bball/bball_base_link, origin xyz=0 0 0.06 rpy=0 0 1.57079
- added joint wam/bball/bball_center_joint: type fixed, parent wam/bball/bball_base_link, child wam/bball/bball_center_link, origin xyz=0 0 0.1 rpy=0 0 0
- joint wam/wam_fixed_joint: origin xyz=0.0 0.0 1.0 rpy=0 0 0 -> xyz=0.0 0.0 0.5 rpy=0 0 0

File: champ_description/urdf/wam_ball.xacro (robot description, xacro)
@@ -34,7 +34,4 @@
 </joint>
 <!-- ArmStuff -->
-<!-- BHand
-<xacro:bhand prefix="wam/bhand" parent_link="wam/wrist_palm_link" xyz="0 0 0.06" rpy="0 0 0"/>
--->
 <!--Ball-->
 <xacro:bball parent_link="wam/wrist_palm_link" prefix="wam/ball" xyz="0 0 0.06" rpy="0 0 0"/>
@@ -135,92 +132,4 @@
     </actuator>
   </transmission>
-<!-- wam/bhand/finger_1/prox_joint -->
-  <transmission name="f1_prox">
-    <type>transmission_interface/SimpleTransmission</type>
-    <joint name="wam/bhand/finger_1/prox_joint">
-      <hardwareInterface>hardware_interface/EffortJointInterface</hardwareInterface>
-    </joint>
-    <actuator name="motor8_1">
-      <hardwareInterface>hardware_interface/EffortJointInterface</hardwareInterface>
-      <mechanicalReduction>1</mechanicalReduction>
-    </actuator>
-  </transmission>
-<!-- wam/bhand/finger_1/med_joint -->
-  <transmission name="f1_med">
-    <type>transmission_interface/SimpleTransmission</type>
-    <joint name="wam/bhand/finger_1/med_joint">
-      <hardwareInterface>hardware_interface/EffortJointInterface</hardwareInterface>
-    </joint>
-    <actuator name="motor8_2">
-      <hardwareInterface>hardware_interface/EffortJointInterface</hardwareInterface>
-      <mechanicalReduction>1</mechanicalReduction>
-    </actuator>
-  </transmission>
-<!-- wam/bhand/finger_1/dist_joint -->
-  <transmission name="f1_dist">
-    <type>transmission_interface/SimpleTransmission</type>
-    <joint name="wam/bhand/finger_1/dist_joint">
-      <hardwareInterface>hardware_interface/EffortJointInterface</hardwareInterface>
-    </joint>
-    <actuator name="motor8_3">
-      <hardwareInterface>hardware_interface/EffortJointInterface</hardwareInterface>
-      <mechanicalReduction>1</mechanicalReduction>
-    </actuator>
-  </transmission>
-<!-- wam/bhand/finger_2/prox_joint -->
-  <transmission name="f2_prox">
-    <type>transmission_interface/SimpleTransmission</type>
-    <joint name="wam/bhand/finger_2/prox_joint">
-      <hardwareInterface>hardware_interface/EffortJointInterface</hardwareInterface>
-    </joint>
-    <actuator name="motor9_1">
-      <hardwareInterface>hardware_interface/EffortJointInterface</hardwareInterface>
-      <mechanicalReduction>1</mechanicalReduction>
-    </actuator>
-  </transmission>
-<!-- wam/bhand/finger_2/med_joint -->
-  <transmission name="f2_med">
-    <type>transmission_interface/SimpleTransmission</type>
-    <joint name="wam/bhand/finger_2/med_joint">
-      <hardwareInterface>hardware_interface/EffortJointInterface</hardwareInterface>
-    </joint>
-    <actuator name="motor9_2">
-      <hardwareInterface>hardware_interface/EffortJointInterface</hardwareInterface>
-      <mechanicalReduction>1</mechanicalReduction>
-    </actuator>
-  </transmission>
-<!-- wam/bhand/finger_2/dist_joint -->
-  <transmission name="f2_dist">
-    <type>transmission_interface/SimpleTransmission</type>
-    <joint name="wam/bhand/finger_2/dist_joint">
-      <hardwareInterface>hardware_interface/EffortJointInterface</hardwareInterface>
-    </joint>
-    <actuator name="motor9_3">
-      <hardwareInterface>hardware_interface/EffortJointInterface</hardwareInterface>
-      <mechanicalReduction>1</mechanicalReduction>
-    </actuator>
-  </transmission>
-<!-- wam/bhand/finger_3/med_joint -->
-  <transmission name="f3_med">
-    <type>transmission_interface/SimpleTransmission</type>
-    <joint name="wam/bhand/finger_3/med_joint">
-      <hardwareInterface>hardware_interface/EffortJointInterface</hardwareInterface>
-    </joint>
-    <actuator name="motor10_1">
-      <hardwareInterface>hardware_interface/EffortJointInterface</hardwareInterface>
-      <mechanicalReduction>1</mechanicalReduction>
-    </actuator>
-  </transmission>
-<!-- wam/bhand/finger_3/dist_joint -->
-  <transmission name="f3_dist">
-    <type>transmission_interface/SimpleTransmission</type>
-    <joint name="wam/bhand/finger_3/dist_joint">
-      <hardwareInterface>hardware_interface/EffortJointInterface</hardwareInterface>
-    </joint>
-    <actuator name="motor10_2">
-      <hardwareInterface>hardware_interface/EffortJointInterface</hardwareInterface>
-      <mechanicalReduction>1</mechanicalReduction>
-    </actuator>
-  </transmission>
 <gazebo>
   <plugin name="gazebo_ros_control" filename="libgazebo_ros_control.so">

File: champ_description/urdf/wam_bhand_powerbot.xacro (robot description, xacro)
@@ -7,10 +7,14 @@
   <!-- Includea all the WAM stuff -->
   <xacro:include filename="$(find champ_description)/urdf/wam/wam_top.urdf.xacro"/>
+<!--
 <link name="cam"/>
-  <!-- Include powerbot -->
+-->
+  <!-- Include powerbot
  <xacro:include filename="$(find champ_description)/urdf/powerbot/powerbot.xacro"/>
+ -->
 <!-- Load kinect from turtlebot_description and position it at origin from asus_cal -->
 <xacro:include filename="$(find champ_description)/urdf/sensors/asus/asus_cal.xacro"/>
 <xacro:include filename="$(find champ_description)/urdf/sensors/asus/asus_xtion_pro.urdf.xacro"/>
+<!--
 <xacro:sensor_asus_xtion_pro parent="cam"/>
 <joint name="cam_joint" type="fixed">
@@ -19,4 +23,5 @@
 	<child link="cam"/>
 </joint>
+-->
 <!-- Kinect stuff
   <xacro:include filename="$(find champ_description)/urdf/asus/asus.xacro"/>
@@ -28,4 +33,5 @@
 <!-- Root link is in the world frame-->
 <link name="world"/>
+<!--
 <joint name="world_fixed_joint" type="fixed">
 <origin xyz="0 0 0" rpy="0 0 0"/>
@@ -33,13 +39,13 @@
 <child link="base_center"/>
 </joint>
+-->
 <!-- ArmStuff -->
-<!-- BHand
+<!-- BHand -->
 <xacro:bhand prefix="wam/bhand" parent_link="wam/wrist_palm_link" xyz="0 0 0.06" rpy="0 0 0"/>
--->
-<!--Ball-->
-<xacro:bball parent_link="wam/wrist_palm_link" prefix="wam/ball" xyz="0 0 0.06" rpy="0 0 0"/>
 <!-- 7-DOF Wam on top of top plate-->
-<xacro:wam_7dof prefix="wam" parent_link="arm_plate" xyz="0.22 0.0 0.05" rpy="0 0 0" />
+<xacro:wam_7dof prefix="wam" parent_link="world" xyz="0.22 0.0 1.0" rpy="0 0 0" />
+<!--
 <xacro:powerbot/>
+-->
 <!--Joint Controllers
 - ARM

File: champ_description/urdf/wam_powerbot.urdf (robot description, URDF)
Before this commit: robot wam_powerbot, 44 links, 43 joints
Links:
- removed link kinect_depth_frame
- removed link kinect_depth_optical_frame
- removed link kinect_link
- removed link kinect_rgb_frame
- removed link kinect_rgb_optical_frame
- removed link left_hubcap
- removed link left_swivel
- removed link left_swivel_hubcap
- removed link left_swivel_support
- removed link left_swivel_wheel
- removed link left_wheel
- removed link right_hubcap
- removed link right_swivel
- removed link right_swivel_hubcap
- removed link right_swivel_support
- removed link right_swivel_wheel
- removed link right_wheel
- added link cam
- added link camera_depth_frame
- added link camera_depth_optical_frame
- added link camera_link, mass 0.170; collision box size=0.0730 0.2760 0.0720; visual mesh filename=package://champ_description/meshes/sensors/xtion_pro_camera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
- added link camera_rgb_frame
- added link camera_rgb_optical_frame
- link base_center: mass 200.0 -> 120.0; geometry collision mesh filename=package://champ_description/meshes/p3dx_meshes/chassis.stl scale=1.01 1.01 1.01; visual mesh filename=package://champ_description/meshes/p3dx_meshes/chassis.stl
- link wam/bhand/finger_1/tip_link: mass 1E-6 -> 0.031377
- link wam/bhand/finger_2/tip_link: mass 1E-6 -> 0.031377
- link wam/bhand/finger_3/tip_link: mass 1E-6 -> 0.031377
Joints:
- removed joint kinect_depth_joint
- removed joint kinect_depth_optical_joint
- removed joint kinect_joint
- removed joint kinect_rgb_joint
- removed joint kinect_rgb_optical_joint
- removed joint left_base_swivel_joint
- removed joint left_base_swivel_support_joint
- removed joint left_hub_joint
- removed joint left_swivel_hubcap_joint
- removed joint left_swivel_wheel_hubcap_joint
- removed joint left_wheel_joint
- removed joint powerbot/world_joint
- removed joint right_base_swivel_joint
- removed joint right_base_swivel_support_joint
- removed joint right_hub_joint
- removed joint right_swivel_hubcap_joint
- removed joint right_swivel_wheel_hubcap_joint
- removed joint right_wheel_joint
- added joint cam_joint: type fixed, parent base_center, child cam, origin xyz=0.351798 0.0081349 0.16 rpy=0.0202643 0.315979 0.0134257
- added joint camera_depth_joint: type fixed, parent camera_rgb_frame, child camera_depth_frame, origin xyz=0 0.027 0 rpy=0 0 0
- added joint camera_depth_optical_joint: type fixed, parent camera_depth_frame, child camera_depth_optical_frame, origin xyz=0 0 0 rpy=-1.570795 0 -1.570795
- added joint camera_joint: type fixed, parent camera_rgb_frame, child camera_link, origin xyz=0 -0.022 0 rpy=0 0 0
- added joint camera_rgb_joint: type fixed, parent cam, child camera_rgb_frame, origin xyz=-0.087 0.0205 0.287 rpy=0 0 0
- added joint camera_rgb_optical_joint: type fixed, parent camera_rgb_frame, child camera_rgb_optical_frame, origin xyz=0 0 0 rpy=-1.570795 0 -1.570795
- added joint world_fixed_joint: type fixed, parent world, child base_center, origin xyz=0 0 0 rpy=0 0 0
