Commit message: added wam_only launch file for gazebo. To Do: - Find a way to rename or remap the joint names to the wam_joint_<num> convention - Fix Powerbot meshes and inertial elements in Mesh lab

File: champ_description/urdf/powerbot/powerbot.urdf (robot description, URDF)
Before this commit: robot powerbot, 15 links, 14 joints
Links:
- removed link back_sonar
- removed link center_hubcap
- removed link center_hubcap2
- removed link center_wheel
- removed link center_wheel2
- removed link front_sonar
- removed link left_hub
- removed link left_wheel_joint
- removed link right_hub
- removed link right_wheel_joint
- removed link swivel
- removed link swivel2
Joints:
- removed joint base_back_joint
- removed joint base_front_joint
- removed joint base_swivel_joint
- removed joint base_swivel_joint2
- removed joint center_wheel_joint
- removed joint center_wheel_joint2
- removed joint left_hub_joint
- removed joint left_wheel_joint
- removed joint right_hub_joint
- removed joint right_wheel_joint
- removed joint swivel_hubcap_joint
- removed joint swivel_hubcap_joint2
- joint base_top_joint: origin xyz=-0.045 0 0.3085 rpy=0 0 0 -> xyz=-0.045 0 0.244 rpy=0 0 0

File: champ_description/urdf/powerbot/powerbot.xacro (robot description, xacro)
@@ -18,5 +18,5 @@
   <xacro:property name="mesh_directory" value="package://champ_description/meshes/p3dx_meshes"/>
   <!--bcz = base_center z value -->
-  <xacro:property name="bcz" value="0.1315"/> <!-- 0.148 -->
+  <xacro:property name="bcz" value="0.067"/> <!-- 0.148 -->
 <!-- Brown arm plate -->
 <link name="arm_plate">
@@ -107,7 +107,7 @@
 	</link>
 	<gazebo reference="base_center">
-		<material>Gazebo/Yellow"</material>
-	</gazebo>
-<!-- Swivel2 -->
+		<material value ="Gazebo/Yellow"/>
+	</gazebo>
+<!-- Swivel2
 	<link name="swivel2">
 		<inertial>
@@ -137,5 +137,4 @@
 	</gazebo>
 	<joint name="base_swivel_joint2" type="continuous">
-		<!--origin xyz="0.045 0 0.055" rpy="0 0 0"/-->
 		<origin xyz="0.045 0 ${bcz - 0.093}" rpy="0 0 0"/>
 		<anchor xyz="0 0 0"/>
@@ -145,5 +144,6 @@
 		<child link="swivel2"/>
 	</joint>
-<!-- Center Wheel + Hubcap -->
+-->
+<!-- Center Wheel + Hubcap
 	<link name="center_hubcap2">
 		<inertial>
@@ -213,5 +213,6 @@
 		<child link="center_hubcap2"/>
 	</joint>
-  <!-- Swivel -->
+ -->
+  <!-- Swivel
 	<link name="swivel">
 		<inertial>
@@ -241,5 +242,4 @@
 	</gazebo>
 	<joint name="base_swivel_joint" type="continuous">
-		<!--origin xyz="0.045 0 0.055" rpy="0 0 0"/-->
 		<origin xyz="0.045 0 ${bcz - 0.093}" rpy="0 0 0"/>
 		<anchor xyz="0 0 0"/>
@@ -249,5 +249,6 @@
 		<child link="swivel"/>
 	</joint>
-<!-- Center Wheel + Hubcap -->
+-->
+<!-- Center Wheel + Hubcap
 	<link name="center_hubcap">
 		<inertial>
@@ -316,5 +317,6 @@
 		<child link="center_hubcap"/>
 	</joint>
-	<!--Wheels-->
+-->
+	<!--Wheels
 	<link name="left_hub">
 		<visual>
@@ -329,5 +331,4 @@
 	</link>
 	<joint name="left_hub_joint" type="fixed">
-		<!--origin xyz="0.1 0.30 0.04" rpy="0 0 0"/-->
 		<origin xyz="0.1 0.30 ${bcz - 0.108}" rpy="0 0 0"/>
 		<parent link="base_center"/>
@@ -369,5 +370,4 @@
 	</gazebo>
 	<joint name="right_hub_joint" type="fixed">
-		<!--origin xyz="0.1 -0.30 0.04" rpy="0 0 0"/-->
 		<origin xyz="0.1 -0.30 ${bcz - 0.108}" rpy="0 0 0"/>
 		<parent link="base_center"/>
@@ -394,5 +394,6 @@
 		<material value="Gazebo/Black"/>
 	</gazebo>
-<!-- Front + Back Sonar -->
+-->
+<!-- Front + Back Sonar
 	<link name="front_sonar">
 		<inertial>
@@ -422,5 +423,4 @@
 	</gazebo>
 	<joint name="base_front_joint" type="fixed">
-		<!--origin xyz="-0.198 0 0.208" rpy="0 0 0"/-->
 		<origin xyz="-0.198 0 ${bcz + 0.06}" rpy="0 0 0"/>
 		<parent link="base_center"/>
@@ -454,9 +454,9 @@
 	</gazebo>
 	<joint name="base_back_joint" type="fixed">
-		<!--origin xyz="0.109 0 0.209" rpy="0 0 0"/-->
 		<origin xyz="0.109 0 ${bcz + 0.061}" rpy="0 0 0"/>
 		<parent link="base_center"/>
 		<child link="back_sonar"/>
 	</joint>
+ -->
 <xacro:macro name="p3at_gazebo_ext">
 <gazebo>

File: champ_description/urdf/wam/wam7_bhand.urdf.xacro (robot description, xacro)
@@ -3,9 +3,9 @@
   xmlns:xacro="http://www.ros.org/wiki/xacro">
   <!-- Includea all the WAM stuff -->
-  <xacro:include filename="$(find champ_description)/urdf/wam_top.urdf.xacro"/>
+  <xacro:include filename="$(find champ_description)/urdf/wam/wam_top.urdf.xacro"/>
   <!-- Root link is in the world frame-->
   <link name="world"/>
   <!-- 7-DOF Wam -->
-  <xacro:wam_7dof prefix="wam" parent_link="world" xyz="0.0 0.0 1.0" rpy="0 0 0" />
+  <xacro:wam_7dof prefix="wam" parent_link="world" xyz="0.0 0.0 0.5" rpy="0 0 0" />
   <!-- BHand -->
   <xacro:bhand prefix="wam/bhand" parent_link="wam/wrist_palm_link" xyz="0 0 0.06" rpy="0 0 1.57079"/>

Commit message: Modified the p3dx_meshes, scaled them to powerbot dimensions using meshlab. Added Wam description and control packages.

File: champ_description/urdf/powerbot/powerbot.urdf (robot description, URDF)
Before this commit: robot powerbot, 3 links, 2 joints
Links:
- link base_center: geometry collision mesh filename=package://champ_description/meshes/p3dx_meshes/chassis.stl; visual mesh filename=package://champ_description/meshes/p3dx_meshes/chassis.stl
- link top_plate: geometry collision mesh filename=package://champ_description/meshes/p3dx_meshes/top.stl; visual mesh filename=package://champ_description/meshes/p3dx_meshes/top.stl

File: champ_description/urdf/wam_powerbot.urdf (robot description, URDF)
Before this commit: robot wam_powerbot, 44 links, 43 joints
Links:
- link base_center: mass None -> 120.0; geometry collision mesh filename=package://champ_description/meshes/p3dx_meshes/chassis.stl; visual mesh filename=package://champ_description/meshes/p3dx_meshes/chassis.stl

Commit message: Fixed powerbot.xacro, changed mesh names, fixed inertias Issue: swivel wheels seem to sink into the base but not the ground. Fix attempt 1: added swivel support meshes so that continuos joint is now between swivels and their supports.

File: champ_description/urdf/powerbot/powerbot.urdf (robot description, URDF)
Before this commit: robot powerbot, 3 links, 2 joints
Links:
- removed link arm_plate
- added link left_hubcap, mass 0.08; collision mesh filename=package://champ_description/meshes/p3dx_meshes/hubcap.stl; visual mesh filename=package://champ_description/meshes/p3dx_meshes/hubcap.stl
- added link left_swivel, mass 0.1; collision mesh filename=package://champ_description/meshes/p3dx_meshes/swivel.stl; visual mesh filename=package://champ_description/meshes/p3dx_meshes/swivel.stl
- added link left_swivel_hubcap, mass 0.01; collision mesh filename=package://champ_description/meshes/p3dx_meshes/center_hubca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; visual mesh filename=package://champ_description/meshes/p3dx_meshes/center_hubca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
- added link left_swivel_support, mass 0.1; collision mesh filename=package://champ_description/meshes/p3dx_meshes/swivel_suppo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; visual mesh filename=package://champ_description/meshes/p3dx_meshes/swivel_suppo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
- added link left_swivel_wheel, mass 0.1; collision cylinder length=0.0422 radius=0.0669; visual mesh filename=package://champ_description/meshes/p3dx_meshes/center_wheel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
- added link left_wheel, mass 1.25; collision cylinder length=0.065 radius=0.1315; visual mesh filename=package://champ_description/meshes/p3dx_meshes/wheel.stl
- added link right_hubcap, mass 0.08; collision mesh filename=package://champ_description/meshes/p3dx_meshes/hubcap.stl; visual mesh filename=package://champ_description/meshes/p3dx_meshes/hubcap.stl
- added link right_swivel, mass 0.1; collision mesh filename=package://champ_description/meshes/p3dx_meshes/swivel.stl; visual mesh filename=package://champ_description/meshes/p3dx_meshes/swivel.stl
- added link right_swivel_hubcap, mass 0.01; collision mesh filename=package://champ_description/meshes/p3dx_meshes/center_hubca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; visual mesh filename=package://champ_description/meshes/p3dx_meshes/center_hubca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
- added link right_swivel_support, mass 0.1; collision mesh filename=package://champ_description/meshes/p3dx_meshes/swivel_suppo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; visual mesh filename=package://champ_description/meshes/p3dx_meshes/swivel_suppo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
- added link right_swivel_wheel, mass 0.1; collision cylinder length=0.0422 radius=0.0669; visual mesh filename=package://champ_description/meshes/p3dx_meshes/center_wheel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
- added link right_wheel, mass 1.25; collision cylinder length=0.065 radius=0.1315; visual mesh filename=package://champ_description/meshes/p3dx_meshes/wheel.stl
- link base_center: mass None -> 120.0
Joints:
- removed joint arm_plate_joint
- added joint left_base_swivel_joint: type continuous, parent left_swivel_support, child left_swivel, origin xyz=0 0 0 rpy=0 0 0, axis 0 0 1, limit effort=100 velocity=100
- added joint left_base_swivel_support_joint: type fixed, parent base_center, child left_swivel_support, origin xyz=-0.215 0.2 -0.14 rpy=0 0 0
- added joint left_hub_joint: type continuous, parent base_center, child left_hubcap, origin xyz=0.1 0.35 -0.0835 rpy=0 0 0, axis 0 1 0, limit effort=100 velocity=100
- added joint left_swivel_hubcap_joint: type continuous, parent left_swivel, child left_swivel_hubcap, origin xyz=-0.036 0 -0.029 rpy=0 0 0, axis 0 1 0, limit effort=100 velocity=100
- added joint left_swivel_wheel_hubcap_joint: type fixed, parent left_swivel_hubcap, child left_swivel_wheel, origin xyz=0 0 0 rpy=0 0 0
- added joint left_wheel_joint: type fixed, parent left_hubcap, child left_wheel, origin xyz=0 0 0 rpy=0 0 0
- added joint right_base_swivel_joint: type continuous, parent right_swivel_support, child right_swivel, origin xyz=0 0 0 rpy=0 0 0, axis 0 0 1, limit effort=100 velocity=100
- added joint right_base_swivel_support_joint: type fixed, parent base_center, child right_swivel_support, origin xyz=-0.215 -0.2 -0.14 rpy=0 0 0
- added joint right_hub_joint: type continuous, parent base_center, child right_hubcap, origin xyz=0.1 -0.35 -0.0835 rpy=0 0 0, axis 0 1 0, limit effort=100 velocity=100
- added joint right_swivel_hubcap_joint: type continuous, parent right_swivel, child right_swivel_hubcap, origin xyz=-0.036 0 -0.029 rpy=0 0 0, axis 0 1 0, limit effort=100 velocity=100
- added joint right_swivel_wheel_hubcap_joint: type fixed, parent right_swivel_hubcap, child right_swivel_wheel, origin xyz=0 0 0 rpy=0 0 0
- added joint right_wheel_joint: type fixed, parent right_hubcap, child right_wheel, origin xyz=0 0 0 rpy=0 0 0
- joint base_top_joint: origin xyz=-0.045 0 0.244 rpy=0 0 0 -> xyz=-0.045 0 0.277 rpy=0 0 0

File: champ_description/urdf/powerbot/powerbot.xacro (robot description, xacro)
@@ -5,12 +5,4 @@
 	xmlns:interface="http://playerstage.sourceforge.net/gazebo/xmlschema/#interface"
 	xmlns:xacro="http://ros.org/wiki/xacro">
- <!-- robot name -->
-  <xacro:macro name="powerbot" params="prefix parent_link xyz rpy">
-    <joint name ="${prefix}/world_joint" type="planar">
-      <parent link="${parent_link}"/>
-      <child link="base_center"/>
-      <origin xyz="${xyz}" rpy="${rpy}"/>
-    </joint>
-  </xacro:macro>
   <!-- Include powerbot wheels -->
   <xacro:include filename="$(find champ_description)/urdf/powerbot/powerbot_wheel.xacro"/>
@@ -19,39 +11,40 @@
   <!--bcz = base_center z value -->
   <xacro:property name="bcz" value="0.067"/> <!-- 0.148 -->
-<!-- Brown arm plate -->
-<link name="arm_plate">
+<!-- Chassis -->
+<link name="base_center">
 	<inertial>
-		<mass value="0.01"/>
-		<origin xyz="2 0 0"/>
-		<inertia ixx="1" ixy="0" ixz="0" iyy="1" iyz="0" izz="1"/>
+	  <mass value="120.0"/>
+	  <origin xyz="-0.045 0 ${bcz}"/>
+	  <inertia ixx="0.4255" ixy="0.0"    ixz="0.0"
+		   		iyy="0.4955" iyz="0.0"
+	          			     izz="0.7441"/>
 	</inertial>
-	<visual>
-		<geometry>
-			<box size="0.45 0.75 0.05"/>
-		</geometry>
-		<origin xyz="0.2 0 0.03" rpy="0 0 0"/>
-		<material name="brown">
-			<color rgba="0.8 0.4 0.3 1"/>
-		</material>
-	</visual>
-	<collision>
-		<origin xyz="0 0 0" rpy="0 0 0"/>
-		<geometry>
-			<box size="0.45 0.75 0.05"/>
-		</geometry>
-	</collision>
-</link>
-<joint name="arm_plate_joint" type="fixed">
-	<parent link="top_plate"/>
-	<child link="arm_plate"/>
-	<origin xyz="0 0 0"/>
-</joint>
+		<visual name="base_visual">
+			<origin xyz="-0.045 0 ${bcz}" rpy="0 0 0"/>
+			<geometry name="pioneer_geom">
+				<mesh filename="${mesh_directory}/chassis.stl"/>
+			</geometry>
+			<material name="ChassisYellow">
+				<color rgba="0.715 0.583 0.210 1.0"/>
+			</material>
+		</visual>
+		<collision>
+			<origin xyz="-0.045 0 ${bcz}" rpy="0 0 0"/>
+			<geometry>
+				<mesh filename="${mesh_directory}/chassis.stl"/>
+			</geometry>
+		</collision>
+	</link>
+	<gazebo reference="base_center">
+		<material value ="Gazebo/Yellow"/>
+	</gazebo>
 <!-- Top -->
 	<joint name="base_top_joint" type="fixed">
 		<!--origin xyz="-0.045 0 0.325" rpy="0 0 0"/-->
-		<origin xyz="-0.045 0 ${bcz + 0.177}" rpy="0 0 0"/>
+		<origin xyz="-0.045 0 0.277" rpy="0 0 0"/>
 		<parent link="base_center"/>
 		<child link="top_plate"/>
 	</joint>
+<!-- Top plate -->
 	<link name="top_plate">
 		<inertial>
@@ -63,14 +56,7 @@
 		</inertial>
 		<visual>
-			<inertial>
-				<mass value="0.01"/>
-				<origin xyz="0 0 0"/>
-				<inertia ixx="1" ixy="0" ixz="0"
-					 iyy="1" iyz="0"
-	 				izz="1"/>
-			</inertial>
 			<origin xyz="0 0 0" rpy="0 0 0"/>
 			<geometry name="top_geom">
-				<mesh filename="${mesh_directory}/top.stl" scale="2 2 2"/>
+				<mesh filename="${mesh_directory}/top.stl"/>
 			</geometry>
 			<material name="TopBlack">
@@ -81,5 +67,5 @@
 			<origin xyz="0 0 0" rpy="0 0 0"/>
 			<geometry>
-				<mesh filename="${mesh_directory}/top.stl" scale="2 2 2"/>
+				<mesh filename="${mesh_directory}/top.stl" />
 			</geometry>
 		</collision>
@@ -88,37 +74,48 @@
 		<material value="Gazebo/Black"/>
 	</gazebo>
-<!-- Chassis -->
-	<link name="base_center">
-		<visual name="base_visual">
-			<origin xyz="-0.045 0 ${bcz}" rpy="0 0 0"/>
-			<geometry name="pioneer_geom">
-				<mesh filename="${mesh_directory}/chassis.stl"  scale="2 2 2"/>
-			</geometry>
-			<material name="ChassisYellow">
-				<color rgba="0.715 0.583 0.210 1.0"/>
-			</material>
-		</visual>
-		<collision>
-			<origin xyz="0 0 0" rpy="0 0 0"/>
-				<geometry>
-					<mesh filename="${mesh_directory}/chassis.stl"  scale="2 2 2"/>
-				</geometry>
-		</collision>
-	</link>
-	<gazebo reference="base_center">
-		<material value ="Gazebo/Yellow"/>
-	</gazebo>
-<!-- Swivel2
-	<link name="swivel2">
-		<inertial>
-			<mass value="0.1"/>
-			<origin xyz="0 0 0"/>
+  <!-- Right Swivel support-->
+	<link name="right_swivel_support">
+		<inertial>
+			<mass value="0.1"/>
+			<origin xyz="0 0 0" rpy="0 0 0"/>
 			<inertia ixx="0.01" ixy="0" ixz="0"
 				 iyy="0.01" iyz="0" izz="0.01"/>
   	 	</inertial>
-	<visual name="base_visual">
-		<origin xyz="-0.26 -0.25 -0.08" rpy="0 0 0"/>
-		<geometry name="pioneer_geom">
-			<mesh filename="${mesh_directory}/swivel.stl" scale="1.5 1.5 1.5"/>
+	<visual name="right_swivel_support_visual">
+		<origin xyz="0 0 0" rpy="0 0 0"/>
+		<geometry name="swivel">
+			<mesh filename="${mesh_directory}/swivel_support.stl" />
+		</geometry>
+		<material name="swivel">
+			<color rgba="0.1 0.1 0.1 1"/>
+		</material>
+	</visual>
+	<collision>
+		<origin xyz="0 0 0" rpy="0 0 0"/>
+		<geometry>
+			<mesh filename="${mesh_directory}/swivel_support.stl" />
+		</geometry>
+	</collision>
+	</link>
+	<gazebo reference="swivel">
+		<material value="Gazebo/Grey"/>
+	</gazebo>
+	<joint name="right_base_swivel_support_joint" type="fixed">
+		<origin xyz="-0.215 -0.2 -0.14" rpy="0 0 0"/>
+		<parent link="base_center"/>
+		<child link="right_swivel_support"/>
+	</joint>
+  <!-- Right Swivel -->
+	<link name="right_swivel">
+		<inertial>
+			<mass value="0.1"/>
+			<origin xyz="0 0 0" rpy="0 0 0"/>
+			<inertia ixx="0.01" ixy="0" ixz="0"
+				 iyy="0.01" iyz="0" izz="0.01"/>
+  	 	</inertial>
+	<visual name="right_swivel_visual">
+		<origin xyz="0 0 0" rpy="0 0 0"/>
+		<geometry name="swivel">
+			<mesh filename="${mesh_directory}/swivel.stl" />
 		</geometry>
 		<material name="swivel">
@@ -129,22 +126,21 @@
 		<origin xyz="0 0 0" rpy="0 0 0"/>
 		<geometry>
-			<mesh filename="${mesh_directory}/swivel.stl" scale="1.5 1.5 1.5"/>
-		</geometry>
-	</collision>
-	</link>
-	<gazebo reference="swivel2">
+			<mesh filename="${mesh_directory}/swivel.stl" />
+		</geometry>
+	</collision>
+	</link>
+	<gazebo reference="swivel">
 		<material value="Gazebo/Grey"/>
 	</gazebo>
-	<joint name="base_swivel_joint2" type="continuous">
-		<origin xyz="0.045 0 ${bcz - 0.093}" rpy="0 0 0"/>
-		<anchor xyz="0 0 0"/>
-    	<limit effort="100" velocity="100" k_velocity="0" />
-    	<joint_properties damping="0.0" friction="0.0" />
-		<parent link="base_center"/>
-		<child link="swivel2"/>
-	</joint>
--->
-<!-- Center Wheel + Hubcap
-	<link name="center_hubcap2">
+	<joint name="right_base_swivel_joint" type="continuous">
+		<origin xyz="0 0 0" rpy="0 0 0"/>
+		<axis xyz="0 0 1"/>
+	    	<limit effort="100" velocity="100" k_velocity="0" />
+	    	<joint_properties damping="0.0" friction="0.0" />
+		<parent link="right_swivel_support"/>
+		<child link="right_swivel"/>
+	</joint>
+<!-- Right swivel Wheel + Hubcap -->
+	<link name="right_swivel_hubcap">
 		<inertial>
 			<mass value="0.01"/>
@@ -153,8 +149,8 @@
 				 iyy="0.015218160428" iyz="-0.000004273467" izz="0.011763977943"/>
   	 	</inertial>
-	<visual name="base_visual">
-		<origin xyz="-0.26 -0.25 -0.08" rpy="0 0 0"/>
+	<visual name="right_swivel_hubcap">
+		<origin xyz="0 0 0" rpy="0 0 0"/>
 		<geometry name="pioneer_geom">
-			<mesh filename="${mesh_directory}/center_hubcap.stl" scale="1.5 1.5 1.5"/>
+			<mesh filename="${mesh_directory}/center_hubcap.stl" />
 		</geometry>
 		<material name="swivel">
@@ -165,21 +161,21 @@
 		<origin xyz="0 0 0" rpy="0 0 0"/>
 		<geometry>
-			<box size="0.05 0.05 0.05"/>
-		</geometry>
-	</collision>
-	</link>
-	<gazebo reference="center_hubcap2">
+			<mesh filename="${mesh_directory}/center_hubcap.stl" />
+		</geometry>
+	</collision>
+	</link>
+	<gazebo reference="swivel_hubcap">
 		<material value="Gazebo/Grey"/>
 	</gazebo>
-	<joint name="swivel_hubcap_joint2" type="continuous">
-		<origin xyz="-0.026 0 -0.016" rpy="0 0 0"/>
+	<joint name="right_swivel_hubcap_joint" type="continuous">
+		<origin xyz="-0.036 0 -0.029" rpy="0 0 0"/>
 		<axis xyz="0 1 0"/>
 		<anchor xyz="0 0 0"/>
     <limit effort="100" velocity="100" k_velocity="0" />
     <joint_properties damping="0.0" friction="0.0" />
-	  <parent link="swivel2"/>
-		<child link="center_wheel2"/>
-	</joint>
-	<link name="center_wheel2">
+	  <parent link="right_swivel"/>
+		<child link="right_swivel_hubcap"/>
+	</joint>
+	<link name="right_swivel_wheel">
 		<inertial>
 			<mass value="0.1"/>
@@ -188,8 +184,8 @@
 				 iyy="0.015218160428" iyz="-0.000004273467" izz="0.011763977943"/>
   	 	</inertial>
-	<visual name="base_visual">
-		<origin xyz="-0.26 -0.25 -0.08" rpy="0 0 0"/>
-		<geometry name="pioneer_geom">
-			<mesh filename="${mesh_directory}/center_wheel.stl" scale="1.5 1.5 1.5"/>
+	<visual name="right_swivel_wheel">
+		<origin xyz="0 0 0" rpy="0 0 0"/>
+		<geometry name="swivel_wheel">
+			<mesh filename="${mesh_directory}/center_wheel.stl" />
 		</geometry>
 		<material name="WheelBlack">
@@ -198,32 +194,62 @@
 	</visual>
 	<collision>
-		<origin xyz="0 0 0" rpy=" 0 0 0"/>
-		<geometry>
-			<mesh filename="${mesh_directory}/center_wheel.stl" scale="1.5 1.5 1.5"/>
-			<cylinder radius="0.0375" length="0.01"/>
-		</geometry>
-	</collision>
-	</link>
-	<gazebo reference="left_hub2">
-		<material value="Gazebo/Yellow"/>
-	</gazebo>
-	<joint name="center_wheel_joint2" type="fixed">
-		<origin xyz="-0.0035 0 -0.001" rpy="0 0 0"/>
-		<parent link="center_wheel2"/>
-		<child link="center_hubcap2"/>
-	</joint>
- -->
-  <!-- Swivel
-	<link name="swivel">
-		<inertial>
-			<mass value="0.1"/>
-			<origin xyz="0 0 0"/>
+		<origin xyz="0 0 0" rpy=" ${-3.1415927/2} 0 0"/>
+		<geometry>
+			<cylinder radius="0.0669" length="0.0422"/>
+		</geometry>
+	</collision>
+	</link>
+	<gazebo reference="swivel_wheel">
+		<material value="Gazebo/Black"/>
+	</gazebo>
+	<joint name="right_swivel_wheel_hubcap_joint" type="fixed">
+		<origin xyz="0 0 0" rpy="0 0 0"/>
+		<parent link="right_swivel_hubcap"/>
+		<child link="right_swivel_wheel"/>
+	</joint>
+  <!-- Left Swivel support-->
+	<link name="left_swivel_support">
+		<inertial>
+			<mass value="0.1"/>
+			<origin xyz="0 0 0" rpy="0 0 0"/>
 			<inertia ixx="0.01" ixy="0" ixz="0"
 				 iyy="0.01" iyz="0" izz="0.01"/>
   	 	</inertial>
-	<visual name="base_visual">
-		<origin xyz="-0.26 0.25 -0.08" rpy="0 0 0"/>
-		<geometry name="pioneer_geom">
-			<mesh filename="${mesh_directory}/swivel.stl" scale="1.5 1.5 1.5"/>
+	<visual name="left_swivel_support_visual">
+		<origin xyz="0 0 0" rpy="0 0 0"/>
+		<geometry name="swivel">
+			<mesh filename="${mesh_directory}/swivel_support.stl" />
+		</geometry>
+		<material name="swivel">
+			<color rgba="0.1 0.1 0.1 1"/>
+		</material>
+	</visual>
+	<collision>
+		<origin xyz="0 0 0" rpy="0 0 0"/>
+		<geometry>
+			<mesh filename="${mesh_directory}/swivel_support.stl" />
+		</geometry>
+	</collision>
+	</link>
+	<gazebo reference="swivel">
+		<material value="Gazebo/Grey"/>
+	</gazebo>
+	<joint name="left_base_swivel_support_joint" type="fixed">
+		<origin xyz="-0.215 0.2 -0.14" rpy="0 0 0"/>
+		<parent link="base_center"/>
+		<child link="left_swivel_support"/>
+	</joint>
+  <!--Left Swivel -->
+	<link name="left_swivel">
+		<inertial>
+			<mass value="0.1"/>
+			<origin xyz="0 0 0" rpy="0 0 0"/>
+			<inertia ixx="0.01" ixy="0" ixz="0"
+				 iyy="0.01" iyz="0" izz="0.01"/>
+  	 	</inertial>
+	<visual name="left_swivel_visual">
+		<origin xyz="0 0 0" rpy="0 0 0"/>
+		<geometry name="swivel">
+			<mesh filename="${mesh_directory}/swivel.stl" />
 		</geometry>
 		<material name="swivel">
@@ -234,5 +260,5 @@
 		<origin xyz="0 0 0" rpy="0 0 0"/>
 		<geometry>
-			<mesh filename="${mesh_directory}/swivel.stl" scale="1.5 1.5 1.5"/>
+			<mesh filename="${mesh_directory}/swivel.stl" />
 		</geometry>
 	</collision>
@@ -241,15 +267,14 @@
 		<material value="Gazebo/Grey"/>
 	</gazebo>
-	<joint name="base_swivel_joint" type="continuous">
-		<origin xyz="0.045 0 ${bcz - 0.093}" rpy="0 0 0"/>
-		<anchor xyz="0 0 0"/>
-    	<limit effort="100" velocity="100" k_velocity="0" />
+	<joint name="left_base_swivel_joint" type="continuous">
+		<origin xyz="0 0 0" rpy="0 0 0"/>
+		<axis xyz="0 0 1"/>
+         <limit effort="100" velocity="100" k_velocity="0" />
     	<joint_properties damping="0.0" friction="0.0" />
-		<parent link="base_center"/>
-		<child link="swivel"/>
-	</joint>
--->
-<!-- Center Wheel + Hubcap
-	<link name="center_hubcap">
+		<parent link="left_swivel_support"/>
+		<child link="left_swivel"/>
+	</joint>
+<!-- left swivel Wheel + Hubcap -->
+	<link name="left_swivel_hubcap">
 		<inertial>
 			<mass value="0.01"/>
@@ -258,8 +283,8 @@
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