Commit message: Temporarily solved swivel wheel problem by changing joints from continuous to fixed. Also did the same to left and right wheels to keep powerbot stationary

File: champ_description/urdf/powerbot/powerbot.urdf (robot description, URDF)
Before this commit: robot powerbot, 14 links, 13 joints
Joints:
- joint left_base_swivel_joint: axis 0 0 1 -> (none); limit effort=100 velocity=100 -> (none); origin xyz=0 0 0 rpy=0 0 0 -> xyz=0 0 -0.04855 rpy=0 0 0; type continuous -> fixed
- joint left_base_swivel_support_joint: origin xyz=-0.215 0.2 -0.14 rpy=0 0 0 -> xyz=-0.215 0.2 -0.091 rpy=0 0 0
- joint left_hub_joint: limit effort=100 velocity=100 -> (none); origin xyz=0.1 0.35 -0.0835 rpy=0 0 0 -> xyz=0.034 0.35 -0.0835 rpy=0 0 0; type continuous -> fixed
- joint right_base_swivel_joint: axis 0 0 1 -> (none); limit effort=100 velocity=100 -> (none); origin xyz=0 0 0 rpy=0 0 0 -> xyz=0 0 -0.04855 rpy=0 0 0; type continuous -> fixed
- joint right_base_swivel_support_joint: origin xyz=-0.215 -0.2 -0.14 rpy=0 0 0 -> xyz=-0.215 -0.2 -0.091 rpy=0 0 0
- joint right_hub_joint: limit effort=100 velocity=100 -> (none); origin xyz=0.1 -0.35 -0.0835 rpy=0 0 0 -> xyz=0.034 -0.35 -0.0835 rpy=0 0 0; type continuous -> fixed

File: champ_description/urdf/powerbot/powerbot.xacro (robot description, xacro)
@@ -88,5 +88,5 @@
 		</geometry>
 		<material name="swivel">
-			<color rgba="0.1 0.1 0.1 1"/>
+			<color rgba="0.9 0.9 0.9 1"/>
 		</material>
 	</visual>
@@ -102,5 +102,5 @@
 	</gazebo>
 	<joint name="right_base_swivel_support_joint" type="fixed">
-		<origin xyz="-0.215 -0.2 -0.14" rpy="0 0 0"/>
+		<origin xyz="-0.215 -0.2 -0.091" rpy="0 0 0"/>
 		<parent link="base_center"/>
 		<child link="right_swivel_support"/>
@@ -133,9 +133,9 @@
 		<material value="Gazebo/Grey"/>
 	</gazebo>
-	<joint name="right_base_swivel_joint" type="continuous">
-		<origin xyz="0 0 0" rpy="0 0 0"/>
-		<axis xyz="0 0 1"/>
+	<joint name="right_base_swivel_joint" type="fixed">
+		<origin xyz="0 0 -0.04855" rpy="0 0 0"/>
+		<!--<axis xyz="0 0 1"/>
 	    	<limit effort="100" velocity="100" k_velocity="0" />
-	    	<joint_properties damping="0.0" friction="0.0" />
+	    	<joint_properties damping="0.0" friction="0.0" />-->
 		<parent link="right_swivel_support"/>
 		<child link="right_swivel"/>
@@ -222,5 +222,5 @@
 		</geometry>
 		<material name="swivel">
-			<color rgba="0.1 0.1 0.1 1"/>
+			<color rgba="0.9 0.9 0.9 1"/>
 		</material>
 	</visual>
@@ -236,5 +236,5 @@
 	</gazebo>
 	<joint name="left_base_swivel_support_joint" type="fixed">
-		<origin xyz="-0.215 0.2 -0.14" rpy="0 0 0"/>
+		<origin xyz="-0.215 0.2 -0.091" rpy="0 0 0"/>
 		<parent link="base_center"/>
 		<child link="left_swivel_support"/>
@@ -267,9 +267,9 @@
 		<material value="Gazebo/Grey"/>
 	</gazebo>
-	<joint name="left_base_swivel_joint" type="continuous">
-		<origin xyz="0 0 0" rpy="0 0 0"/>
-		<axis xyz="0 0 1"/>
+	<joint name="left_base_swivel_joint" type="fixed">
+		<origin xyz="0 0 -0.04855" rpy="0 0 0"/>
+	<!--	<axis xyz="0 0 1"/>
          <limit effort="100" velocity="100" k_velocity="0" />
-    	<joint_properties damping="0.0" friction="0.0" />
+    	<joint_properties damping="0.0" friction="0.0" />-->
 		<parent link="left_swivel_support"/>
 		<child link="left_swivel"/>
@@ -366,9 +366,9 @@
 	      </collision>
 	</link>
-	<joint name="left_hub_joint" type="continuous">
-		<origin xyz="0.1 0.35 -0.0835" rpy="0 0 0"/>
-	        <anchor xyz="0 0 0"/>
+	<joint name="left_hub_joint" type="fixed">
+		<origin xyz="0.034 0.35 -0.0835" rpy="0 0 0"/>
+	        <!--<anchor xyz="0 0 0"/>
 	        <limit effort="100" velocity="100" />
-	        <joint_properties damping="0.0" friction="0.0" />
+	        <joint_properties damping="0.0" friction="0.0" />-->
 		<parent link="base_center"/>
 		<child link="left_hubcap"/>
@@ -430,9 +430,9 @@
 	      </collision>
 	</link>
-	<joint name="right_hub_joint" type="continuous">
-		<origin xyz="0.1 -0.35 -0.0835" rpy="0 0 0"/>
-	        <anchor xyz="0 0 0"/>
+	<joint name="right_hub_joint" type="fixed">
+		<origin xyz="0.034 -0.35 -0.0835" rpy="0 0 0"/>
+	        <!--<anchor xyz="0 0 0"/>
 	        <limit effort="100" velocity="100" />
-	        <joint_properties damping="0.0" friction="0.0" />
+	        <joint_properties damping="0.0" friction="0.0" />-->
 		<parent link="base_center"/>
 		<child link="right_hubcap"/>
@@ -470,45 +470,4 @@
 		<material value="Gazebo/Black"/>
 	</gazebo>
-<!--Wheels
-	<link name="right_hub">
-		<visual>
-			<origin xyz="0 0 0" rpy="0 0 0"/>
-			<geometry>
-				<mesh filename="${mesh_directory}/right_hubcap.stl" scale="1.5 1.5 1.5"/>
-			</geometry>
-			<material name="HubcapWhite">
-				<color rgba="1.0 1.0 1.0 1.0"/>
-			</material>
-		</visual>
-	</link>
-	<gazebo reference="right_hub">
-		<material value="Gazebo/Yellow"/>
-	</gazebo>
-	<joint name="right_hub_joint" type="fixed">
-		<origin xyz="0.1 -0.30 ${bcz - 0.108}" rpy="0 0 0"/>
-		<parent link="base_center"/>
-		<child link="right_hub"/>
-		<axis xyz="0 1 0"/>
-	</joint>
-	<link name="right_wheel_joint">
-		<visual>
-			<origin xyz="0 0 0" rpy="0 0 0"/>
-			<geometry>
-				<mesh filename="${mesh_directory}/right_wheel.stl" scale="1.5 1.5 1.5"/>
-			</geometry>
-			<material name="WheelBlack">
-				<color rgba="0.117 0.117 0.117 1"/>
-			</material>
-		</visual>
-	</link>
-	<joint name="right_wheel_joint" type="fixed">
-		<origin xyz="0 0 0" rpy="0 0 0"/>
-		<parent link="right_hub"/>
-		<child link="right_wheel_joint"/>
-	</joint>
-	<gazebo reference="right_wheel_joint">
-		<material value="Gazebo/Black"/>
-	</gazebo>
--->
 <!-- Front + Back Sonar
 	<link name="front_sonar">

Commit message: Added brown top link

File: champ_description/urdf/powerbot/powerbot.urdf (robot description, URDF)
Before this commit: robot powerbot, 14 links, 13 joints
Links:
- added link arm_plate, mass 0.01; collision box size=0.45 0.75 0.05; visual box size=0.45 0.75 0.05
Joints:
- added joint arm_plate_joint: type fixed, parent top_plate, child arm_plate, origin xyz=0 0 0

File: champ_description/urdf/powerbot/powerbot.xacro (robot description, xacro)
@@ -11,4 +11,32 @@
   <!--bcz = base_center z value -->
   <xacro:property name="bcz" value="0.067"/> <!-- 0.148 -->
+<!-- Brown arm plate -->
+<link name="arm_plate">
+	<inertial>
+		<mass value="0.01"/>
+		<origin xyz="0.2 0 0.03" rpy="0 0 0"/>
+		<inertia ixx="1" ixy="0" ixz="0" iyy="1" iyz="0" izz="1"/>
+	</inertial>
+	<visual>
+		<geometry>
+			<box size="0.45 0.75 0.05"/>
+		</geometry>
+		<origin xyz="0.2 0 0.03" rpy="0 0 0"/>
+		<material name="brown">
+			<color rgba="0.8 0.4 0.3 1"/>
+		</material>
+	</visual>
+	<collision>
+		<origin xyz="0.2 0 0.03" rpy="0 0 0"/>
+		<geometry>
+			<box size="0.45 0.75 0.05"/>
+		</geometry>
+	</collision>
+</link>
+<joint name="arm_plate_joint" type="fixed">
+	<parent link="top_plate"/>
+	<child link="arm_plate"/>
+	<origin xyz="0 0 0"/>
+</joint>
 <!-- Chassis -->
 <link name="base_center">
@@ -334,5 +362,5 @@
 	</collision>
 	</link>
-	<gazebo reference="swivel_wheel">
+	<gazebo reference="right_wheel">
 		<material value="Gazebo/Black"/>
 	</gazebo>

Commit message: Fixed swivel wheel problem by increasing mass to values x  >= 1 instead of 0 <= x <= 1 Issues: - Wam collides with chassis (collisions are failing here) - Bhand still explodes when controller is started. 	- Try Changing joint limits since the BHand 	  joints may be starting outside joint limits 	- Tune PID params make sure values aren't too large.

File: champ_description/urdf/powerbot/powerbot.urdf (robot description, URDF)
Before this commit: robot powerbot, 15 links, 14 joints
Links:
- link left_swivel: mass 0.1 -> 2.0
- link left_swivel_wheel: mass 0.1 -> 2.0; geometry collision cylinder length=0.0422 radius=0.0468; visual mesh filename=package://champ_description/meshes/p3dx_meshes/center_wheel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
- link left_wheel: mass 1.25 -> 5.25
- link right_swivel: mass 0.1 -> 2.0
- link right_swivel_wheel: mass 0.1 -> 2.0; geometry collision cylinder length=0.0422 radius=0.0468; visual mesh filename=package://champ_description/meshes/p3dx_meshes/center_wheel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
- link right_wheel: mass 1.25 -> 5.25
Joints:
- joint left_base_swivel_joint: axis (none) -> 0 0 1; limit (none) -> effort=100 velocity=100; type fixed -> continuous
- joint left_hub_joint: limit (none) -> effort=100 velocity=100; type fixed -> continuous
- joint right_base_swivel_joint: axis (none) -> 0 0 1; limit (none) -> effort=100 velocity=100; type fixed -> continuous
- joint right_hub_joint: limit (none) -> effort=100 velocity=100; type fixed -> continuous

File: champ_description/urdf/powerbot/powerbot.xacro (robot description, xacro)
@@ -145,8 +145,8 @@
 	<link name="right_swivel">
 		<inertial>
-			<mass value="0.1"/>
-			<origin xyz="0 0 0" rpy="0 0 0"/>
-			<inertia ixx="0.01" ixy="0" ixz="0"
-				 iyy="0.01" iyz="0" izz="0.01"/>
+			<mass value="2.0"/>
+			<origin xyz="0 0 0" rpy="0 0 0"/>
+			<inertia ixx="0.001" ixy="0" ixz="0"
+				 iyy="0.001" iyz="0" izz="0.001"/>
   	 	</inertial>
 	<visual name="right_swivel_visual">
@@ -169,9 +169,9 @@
 		<material value="Gazebo/Grey"/>
 	</gazebo>
-	<joint name="right_base_swivel_joint" type="fixed">
+	<joint name="right_base_swivel_joint" type="continuous">
 		<origin xyz="0 0 -0.04855" rpy="0 0 0"/>
-		<!--<axis xyz="0 0 1"/>
+		<axis xyz="0 0 1"/>
 	    	<limit effort="100" velocity="100" k_velocity="0" />
-	    	<joint_properties damping="0.0" friction="0.0" />-->
+	    	<joint_properties damping="7.0" friction="0.7" />
 		<parent link="right_swivel_support"/>
 		<child link="right_swivel"/>
@@ -182,6 +182,6 @@
 			<mass value="0.01"/>
 			<origin xyz="0 0 0"/>
-			<inertia ixx="0.012411765597" ixy="-0.000711733678" ixz="0.00050272983"
-				 iyy="0.015218160428" iyz="-0.000004273467" izz="0.011763977943"/>
+			<inertia ixx="0.00012411765597" ixy="0.0" ixz="0.0"
+				 iyy="0.00015218160428" iyz="0.0" izz="0.00011763977943"/>
   	 	</inertial>
 	<visual name="right_swivel_hubcap">
@@ -209,5 +209,5 @@
 		<anchor xyz="0 0 0"/>
     <limit effort="100" velocity="100" k_velocity="0" />
-    <joint_properties damping="7.0" friction="0.0" />
+    <joint_properties damping="7.0" friction="0.7" />
 	  <parent link="right_swivel"/>
 		<child link="right_swivel_hubcap"/>
@@ -215,8 +215,8 @@
 	<link name="right_swivel_wheel">
 		<inertial>
-			<mass value="0.1"/>
-			<origin xyz="0 0 0"/>
-			<inertia ixx="0.012411765597" ixy="-0.000711733678" ixz="0.00050272983"
-				 iyy="0.015218160428" iyz="-0.000004273467" izz="0.011763977943"/>
+			<mass value="2.0"/>
+			<origin xyz="0 0 0"/>
+			<inertia ixx="0.00012411765597" ixy="0.0" ixz="0.0"
+				 iyy="0.00015218160428" iyz="0.0" izz="0.00011763977943"/>
   	 	</inertial>
 	<visual name="right_swivel_wheel">
@@ -232,5 +232,5 @@
 		<origin xyz="0 0 0" rpy=" ${-3.1415927/2} 0 0"/>
 		<geometry>
-			<cylinder radius="0.0669" length="0.0422"/>
+			<cylinder radius="0.0468" length="0.0422"/>
 		</geometry>
 	</collision>
@@ -279,8 +279,8 @@
 	<link name="left_swivel">
 		<inertial>
-			<mass value="0.1"/>
-			<origin xyz="0 0 0" rpy="0 0 0"/>
-			<inertia ixx="0.01" ixy="0" ixz="0"
-				 iyy="0.01" iyz="0" izz="0.01"/>
+			<mass value="2.0"/>
+			<origin xyz="0 0 0" rpy="0 0 0"/>
+			<inertia ixx="0.001" ixy="0" ixz="0"
+				 iyy="0.001" iyz="0" izz="0.001"/>
   	 	</inertial>
 	<visual name="left_swivel_visual">
@@ -303,9 +303,9 @@
 		<material value="Gazebo/Grey"/>
 	</gazebo>
-	<joint name="left_base_swivel_joint" type="fixed">
+	<joint name="left_base_swivel_joint" type="continuous">
 		<origin xyz="0 0 -0.04855" rpy="0 0 0"/>
-	<!--	<axis xyz="0 0 1"/>
+		<axis xyz="0 0 1"/>
          <limit effort="100" velocity="100" k_velocity="0" />
-    	<joint_properties damping="0.0" friction="0.0" />-->
+    	<joint_properties damping="7.0" friction="0.7" />
 		<parent link="left_swivel_support"/>
 		<child link="left_swivel"/>
@@ -316,6 +316,6 @@
 			<mass value="0.01"/>
 			<origin xyz="0 0 0"/>
-			<inertia ixx="0.012411765597" ixy="-0.000711733678" ixz="0.00050272983"
-				 iyy="0.015218160428" iyz="-0.000004273467" izz="0.011763977943"/>
+			<inertia ixx="0.00012411765597" ixy="0.0" ixz="0.0"
+				 iyy="0.00015218160428" iyz="0.0" izz="0.00011763977943"/>
   	 	</inertial>
 	<visual name="left_swivel_hubcap">
@@ -343,5 +343,5 @@
 		<anchor xyz="0 0 0"/>
     <limit effort="100" velocity="100" k_velocity="0" />
-    <joint_properties damping="7.0" friction="0.0" />
+    <joint_properties damping="7.0" friction="0.7" />
 	  <parent link="left_swivel"/>
 		<child link="left_swivel_hubcap"/>
@@ -349,8 +349,8 @@
 	<link name="left_swivel_wheel">
 		<inertial>
-			<mass value="0.1"/>
-			<origin xyz="0 0 0"/>
-			<inertia ixx="0.012411765597" ixy="-0.000711733678" ixz="0.00050272983"
-				 iyy="0.015218160428" iyz="-0.000004273467" izz="0.011763977943"/>
+			<mass value="2.0"/>
+			<origin xyz="0 0 0"/>
+			<inertia ixx="0.00012411765597" ixy="0.0" ixz="0.0"
+				 iyy="0.00015218160428" iyz="0.0" izz="0.00011763977943"/>
   	 	</inertial>
 	<visual name="left_swivel_wheel">
@@ -366,5 +366,5 @@
 		<origin xyz="0 0 0" rpy=" ${-3.1415927/2} 0 0"/>
 		<geometry>
-			<cylinder radius="0.0669" length="0.0422"/>
+			<cylinder radius="0.0468" length="0.0422"/>
 		</geometry>
 	</collision>
@@ -402,9 +402,9 @@
 	      </collision>
 	</link>
-	<joint name="left_hub_joint" type="fixed">
+	<joint name="left_hub_joint" type="continuous">
 		<origin xyz="0.084 0.35 -0.0835" rpy="0 0 0"/>
-	        <!--<anchor xyz="0 0 0"/>
+	        <anchor xyz="0 0 0"/>
 	        <limit effort="100" velocity="100" />
-	        <joint_properties damping="0.0" friction="0.0" />-->
+	        <joint_properties damping="7.0" friction="2.0" />
 		<parent link="base_center"/>
 		<child link="left_hubcap"/>
@@ -413,5 +413,5 @@
 	<link name="left_wheel">
 	      <inertial>
-		<mass value="1.25"/>
+		<mass value="5.25"/>
 		<origin xyz="0 0 0"/>
 		<inertia ixx="0.012411765597" ixy="0" ixz="0"
@@ -466,9 +466,9 @@
 	      </collision>
 	</link>
-	<joint name="right_hub_joint" type="fixed">
+	<joint name="right_hub_joint" type="continuous">
 		<origin xyz="0.084 -0.35 -0.0835" rpy="0 0 0"/>
-	        <!--<anchor xyz="0 0 0"/>
+	        <anchor xyz="0 0 0"/>
 	        <limit effort="100" velocity="100" />
-	        <joint_properties damping="0.0" friction="0.0" />-->
+	        <joint_properties damping="7.0" friction="2.0" />
 		<parent link="base_center"/>
 		<child link="right_hubcap"/>
@@ -477,5 +477,5 @@
 	<link name="right_wheel">
 	      <inertial>
-		<mass value="1.25"/>
+		<mass value="5.25"/>
 		<origin xyz="0 0 0"/>
 		<inertia ixx="0.012411765597" ixy="0" ixz="0"

File: champ_description/urdf/wam_powerbot.urdf (robot description, URDF)
Before this commit: robot wam_powerbot, 44 links, 43 joints
Links:
- link base_center: mass 120.0 -> 200.0
- link left_wheel: mass 1.25 -> 10.25
- link right_wheel: mass 1.25 -> 10.25
Joints:
- joint left_hub_joint: limit (none) -> effort=100 velocity=100; type fixed -> continuous
- joint right_hub_joint: limit (none) -> effort=100 velocity=100; type fixed -> continuous

File: champ_description/urdf/wam_powerbot.xacro (robot description, xacro)
@@ -19,5 +19,5 @@
 <!-- ArmStuff -->
 <!-- BHand -->
-<xacro:bhand prefix="wam/bhand" parent_link="wam/wrist_palm_link" xyz="0 0 0.1" rpy="0 0 0"/>
+<xacro:bhand prefix="wam/bhand" parent_link="wam/wrist_palm_link" xyz="0 0 0.06" rpy="0 0 0"/>
 <!-- 7-DOF Wam on top of top plate-->
 <xacro:wam_7dof prefix="wam" parent_link="arm_plate" xyz="0.22 0.0 0.05" rpy="0 0 0" />

Commit message: Fixed Jumping links in gazebo. Issues: - Missing differential drive controller for powerbot wheels - PID parameters need tuning but not displaying in rqt_dynamic_reconfigure

File: champ_description/urdf/powerbot/powerbot.urdf (robot description, URDF)
Before this commit: robot powerbot, 15 links, 14 joints
Joints:
- joint left_base_swivel_joint: limit effort=100 velocity=100 -> (none)
- joint left_hub_joint: limit effort=100 velocity=100 -> (none)
- joint left_swivel_hubcap_joint: limit effort=100 velocity=100 -> (none)
- joint right_base_swivel_joint: limit effort=100 velocity=100 -> (none)
- joint right_hub_joint: limit effort=100 velocity=100 -> (none)
- joint right_swivel_hubcap_joint: limit effort=100 velocity=100 -> (none)

File: champ_description/urdf/powerbot/powerbot.xacro (robot description, xacro)
@@ -172,6 +172,5 @@
 		<origin xyz="0 0 -0.04855" rpy="0 0 0"/>
 		<axis xyz="0 0 1"/>
-	    	<limit effort="100" velocity="100" k_velocity="0" />
-	    	<joint_properties damping="7.0" friction="0.7" />
+	    	<joint_properties damping="9.0" />
 		<parent link="right_swivel_support"/>
 		<child link="right_swivel"/>
@@ -208,6 +207,5 @@
 		<axis xyz="0 1 0"/>
 		<anchor xyz="0 0 0"/>
-    <limit effort="100" velocity="100" k_velocity="0" />
-    <joint_properties damping="7.0" friction="0.7" />
+    <joint_properties damping="9.0" />
 	  <parent link="right_swivel"/>
 		<child link="right_swivel_hubcap"/>
@@ -234,4 +232,12 @@
 			<cylinder radius="0.0468" length="0.0422"/>
 		</geometry>
+		      <surface>
+			<friction>
+			  <ode>
+			    <mu>0.8</mu>
+			    <mu2>0.8</mu2>
+			  </ode>
+			</friction>
+		      </surface>
 	</collision>
 	</link>
@@ -306,6 +312,5 @@
 		<origin xyz="0 0 -0.04855" rpy="0 0 0"/>
 		<axis xyz="0 0 1"/>
-         <limit effort="100" velocity="100" k_velocity="0" />
-    	<joint_properties damping="7.0" friction="0.7" />
+    	<joint_properties damping="9.0" />
 		<parent link="left_swivel_support"/>
 		<child link="left_swivel"/>
@@ -342,6 +347,5 @@
 		<axis xyz="0 1 0"/>
 		<anchor xyz="0 0 0"/>
-    <limit effort="100" velocity="100" k_velocity="0" />
-    <joint_properties damping="7.0" friction="0.7" />
+    <joint_properties damping="9.0" />
 	  <parent link="left_swivel"/>
 		<child link="left_swivel_hubcap"/>
@@ -368,4 +372,12 @@
 			<cylinder radius="0.0468" length="0.0422"/>
 		</geometry>
+		      <surface>
+			<friction>
+			  <ode>
+			    <mu>0.8</mu>
+			    <mu2>0.8</mu2>
+			  </ode>
+			</friction>
+		      </surface>
 	</collision>
 	</link>
@@ -405,6 +417,5 @@
 		<origin xyz="0.084 0.35 -0.0835" rpy="0 0 0"/>
 	        <anchor xyz="0 0 0"/>
-	        <limit effort="100" velocity="100" />
-	        <joint_properties damping="7.0" friction="2.0" />
+	        <joint_properties damping="9.0"  />
 		<parent link="base_center"/>
 		<child link="left_hubcap"/>
@@ -432,4 +443,12 @@
 		  <cylinder radius="0.1315" length="0.065"/>
 		</geometry>
+		      <surface>
+			<friction>
+			  <ode>
+			    <mu>0.8</mu>
+			    <mu2>0.8</mu2>
+			  </ode>
+			</friction>
+		      </surface>
 	      </collision>
 	</link>
@@ -469,6 +488,5 @@
 		<origin xyz="0.084 -0.35 -0.0835" rpy="0 0 0"/>
 	        <anchor xyz="0 0 0"/>
-	        <limit effort="100" velocity="100" />
-	        <joint_properties damping="7.0" friction="2.0" />
+	        <joint_properties damping="9.0"  />
 		<parent link="base_center"/>
 		<child link="right_hubcap"/>
@@ -496,4 +514,12 @@
 		  <cylinder radius="0.1315" length="0.065"/>
 		</geometry>
+		      <surface>
+			<friction>
+			  <ode>
+			    <mu>0.8</mu>
+			    <mu2>0.8</mu2>
+			  </ode>
+			</friction>
+		      </surface>
 	      </collision>
 	</link>

File: champ_description/urdf/wam/hand.urdf.xacro (robot description, xacro)
@@ -73,5 +73,5 @@
         <mass value="0.50573" />
         <inertia
-          ixx="3.8374e-005" ixy="-5.604e-008"  ixz="-4.2034e-005"
+          ixx="0.00038374" ixy="-5.604e-008"  ixz="-4.2034e-005"
                            iyy="0.00022405"   iyz="1.3283e-007"
                                               izz="0.00020045" />
@@ -149,7 +149,7 @@
         <mass value="0.14109" />
         <inertia
-          ixx="4.872e-006" ixy="1.7103e-006"  ixz="3.4041e-008"
-                           iyy="7.6588e-005"  iyz="2.3133e-008"
-                                              izz="7.7733e-005" />
+          ixx="0.04872" ixy="1.7103e-006"  ixz="3.4041e-008"
+                           iyy="0.076588"  iyz="2.3133e-008"
+                                              izz="0.077733" />
       </inertial>
       <visual>
@@ -188,7 +188,7 @@
         <mass value="0.062139" />
         <inertia
-          ixx="4.872e-006" ixy="1.7103e-006"  ixz="3.4041e-008"
-                           iyy="7.6588e-005"  iyz="2.3133e-008"
-                                              izz="7.7733e-005" />
+          ixx="0.04872" ixy="1.7103e-006"  ixz="3.4041e-008"
+                           iyy="0.07658"  iyz="2.3133e-008"
+                                              izz="0.077733" />
       </inertial>
       <visual>
@@ -227,7 +227,7 @@
         <mass value="0.041377" />
         <inertia
-          ixx="3.1582e-006" ixy="1.4308e-006"  ixz="1.0106e-007"
-                           iyy="3.8376e-005"   iyz="0"
-                                              izz="3.7275e-005" />
+          ixx="0.031582" ixy="1.4308e-006"  ixz="1.0106e-007"
+                           iyy="0.03837"   iyz="0"
+                                              izz="0.037275" />
       </inertial>
       <visual>
@@ -256,9 +256,9 @@
     <link name="${prefix}/tip_link">
       <inertial>
-        <mass value="1E-6" />
-        <inertia
-          ixx="1E-6" ixy="0"    ixz="0"
-                     iyy="1E-6" iyz="0"
-                                izz="1E-6" />
+        <mass value="0.031377" />
+        <inertia
+          ixx="0.0731582" ixy="1.4308e-006"  ixz="1.0106e-007"
+                           iyy="0.07837"   iyz="0"
+                                              izz="0.07275" />
       </inertial>
     </link>
