Commit message: Working differential drive controller. powerbot.xacro is now split into powerbot_wheel.xacro and powerbot_swivel_wheel.xacro
    Issues:
                - Powerbot refuses to be stationary.
                - Suspects: inertial tensor matrices, swivel wheels, joint friction?
                - Fix holy collisions (in progress).
                - Need to spawn urdf in home position.
                - Fix robot tf tree for use with Rviz and Moveit!

File: champ_description/urdf/powerbot/pioneer3dx_wheel.xacro (robot description, xacro)
@@ -4,46 +4,48 @@
   <!-- Properties (Constants) -->
   <xacro:property name="M_PI" value="3.14159"/>
+  <!-- where to find all meshes -->
+<xacro:property name="mesh_directory" value="package://champ_description/meshes/p3dx_meshes"/>
   <!-- Right/Left Hubcap + Wheel -->
-  <xacro:macro name="p3dx_wheel" params="suffix parent reflect">
-    <link name="p3dx_${suffix}_wheel">
+  <xacro:macro name="powerbot_wheel" params="suffix parent reflect">
+    <link name="powerbot_${suffix}_wheel">
       <inertial>
-        <mass value="0.5"/>
-        <origin xyz="0 0 0"/>
-        <inertia ixx="0.012411765597" ixy="0" ixz="0"
-                 iyy="0.015218160428" iyz="0" izz="0.011763977943"/>
-      </inertial>
-      <visual>
-        <origin xyz="0 0 0" rpy="0 0 0"/>
-        <geometry name="pioneer_geom">
-          <mesh filename="package://p2os_urdf/meshes/p3dx_meshes/${suffix}_wheel.stl"/>
-        </geometry>
-        <material name="WheelBlack">
-          <color rgba="0.117 0.117 0.117 1"/>
-        </material>
-      </visual>
-      <collision>
-        <origin xyz="0 0 0" rpy="${-3.1415927/2} 0 0"/>
-        <geometry>
-          <cylinder radius="0.09" length="0.04"/>
-        </geometry>
-      </collision>
+	<mass value="5.25"/>
+		<origin xyz="0 0 0"/>
+		<inertia ixx="0.012411765597" ixy="0" ixz="0"
+		         iyy="0.015218160428" iyz="0" izz="0.011763977943"/>
+	      </inertial>
+		<visual>
+			<origin xyz="0 0 0" rpy="0 0 0"/>
+			<geometry>
+				<mesh filename="${mesh_directory}/wheel.stl" />
+			</geometry>
+			<material name="WheelBlack">
+				<color rgba="0.117 0.117 0.117 1"/>
+			</material>
+		</visual>
+	<collision>
+		<origin xyz="0 0 0" rpy="${-3.1415927/2} 0 0"/>
+		<geometry>
+		  <cylinder radius="0.133" length="0.065"/>
+		</geometry>
+	</collision>
     </link>
     <joint name="base_${suffix}_hubcap_joint" type="fixed">
       <origin xyz="0 0 0" rpy="0 0 0"/>
-      <parent link="p3dx_${suffix}_wheel"/>
-      <child link="p3dx_${suffix}_hubcap"/>
+      <parent link="powerbot_${suffix}_wheel"/>
+      <child link="powerbot_${suffix}_hubcap"/>
     </joint>
-    <link name="p3dx_${suffix}_hubcap">
-      <inertial>
-        <mass value="0.01"/>
-        <origin xyz="0 0 0"/>
-        <inertia ixx="0.012411765597" ixy="0" ixz="0"
-                 iyy="0.015218160428" iyz="0" izz="0.011763977943"/>
-      </inertial>
-      <visual>
-        <origin xyz="0 0 0" rpy="0 0 0"/>
-        <geometry name="pioneer_geom">
-          <mesh filename="package://p2os_urdf/meshes/p3dx_meshes/${suffix}_hubcap.stl"/>
-        </geometry>
+    <link name="powerbot_${suffix}_hubcap">
+	      <inertial>
+		<mass value="0.08"/>
+		<origin xyz="0 0 0"/>
+		<inertia ixx="0.012411765597" ixy="0" ixz="0"
+		         iyy="0.015218160428" iyz="0" izz="0.011763977943"/>
+	      </inertial>
+		<visual>
+			<origin xyz="0 0 0" rpy="0 0 0"/>
+			<geometry>
+				<mesh filename="${mesh_directory}/hubcap.stl"/>
+			</geometry>
         <material name="HubcapYellow">
           <color rgba="1.0 0.811 0.151 1.0"/>
@@ -62,12 +64,12 @@
       <limit effort="100" velocity="100" />
       <joint_properties damping="0.0" friction="0.0" />
-      <origin xyz="0 ${reflect*0.158} 0.091" rpy="0 0 0"/>
-      <parent link="base_link"/>
-      <child link="p3dx_${suffix}_wheel"/>
+      <origin xyz="0.084 ${reflect*0.35} -0.0835" rpy="0 0 0"/>
+      <parent link="base_center"/>
+      <child link="powerbot_${suffix}_wheel"/>
     </joint>
-    <gazebo reference="p3dx_${suffix}_hubcap">
+    <gazebo reference="powerbot_${suffix}_hubcap">
       <material value="Gazebo/Yellow"/>
     </gazebo>
-    <gazebo reference="p3dx_${suffix}_wheel">
+    <gazebo reference="powerbot_${suffix}_wheel">
       <material value="Gazebo/Black"/>
       <mu1>0.5</mu1>

File: champ_description/urdf/powerbot/powerbot.xacro (robot description, xacro)
@@ -15,4 +15,6 @@
   <!-- Include powerbot wheels -->
   <xacro:include filename="$(find champ_description)/urdf/powerbot/powerbot_wheel.xacro"/>
+  <!-- Include powerbot swivel wheels -->
+  <xacro:include filename="$(find champ_description)/urdf/powerbot/powerbot_swivel_wheel.xacro"/>
   <!-- where to find all meshes -->
   <xacro:property name="mesh_directory" value="package://champ_description/meshes/p3dx_meshes"/>
@@ -61,7 +63,7 @@
 				<mesh filename="${mesh_directory}/chassis.stl"/>
 			</geometry>
-			<material name="ChassisYellow">
-				<color rgba="0.715 0.583 0.210 1.0"/>
-			</material>
+	<material name="ChassisRed">
+		<color rgba="0.8 0.0 0.0 1.0"/>
+	</material>
 		</visual>
 		<collision>
@@ -73,5 +75,5 @@
 	</link>
 	<gazebo reference="base_center">
-		<material value ="Gazebo/Yellow"/>
+		 <material>Gazebo/Red</material>
 	</gazebo>
 <!-- Top -->
@@ -110,426 +112,8 @@
 		<material value="Gazebo/Black"/>
 	</gazebo>
-  <!-- Right Swivel support-->
-	<link name="right_swivel_support">
-		<inertial>
-			<mass value="0.1"/>
-			<origin xyz="0 0 0" rpy="0 0 0"/>
-			<inertia ixx="0.01" ixy="0" ixz="0"
-				 iyy="0.01" iyz="0" izz="0.01"/>
-  	 	</inertial>
-	<visual name="right_swivel_support_visual">
-		<origin xyz="0 0 0" rpy="0 0 0"/>
-		<geometry name="swivel">
-			<mesh filename="${mesh_directory}/swivel_support.stl" />
-		</geometry>
-		<material name="swivel">
-			<color rgba="0.9 0.9 0.9 1"/>
-		</material>
-	</visual>
-	<collision>
-		<origin xyz="0 0 0" rpy="0 0 0"/>
-		<geometry>
-			<mesh filename="${mesh_directory}/swivel_support.stl" scale= "1.005 1.005 1.005"/>
-		</geometry>
-	</collision>
-	</link>
-	<gazebo reference="swivel">
-		<material value="Gazebo/Grey"/>
-	</gazebo>
-	<joint name="right_base_swivel_support_joint" type="fixed">
-		<origin xyz="-0.215 -0.2 -0.0915" rpy="0 0 0"/>
-		<parent link="base_center"/>
-		<child link="right_swivel_support"/>
-	</joint>
-  <!-- Right Swivel -->
-	<link name="right_swivel">
-		<inertial>
-			<mass value="2.0"/>
-			<origin xyz="0 0 0" rpy="0 0 0"/>
-			<inertia ixx="0.001" ixy="0" ixz="0"
-				 iyy="0.001" iyz="0" izz="0.001"/>
-  	 	</inertial>
-	<visual name="right_swivel_visual">
-		<origin xyz="0 0 0" rpy="0 0 0"/>
-		<geometry name="swivel">
-			<mesh filename="${mesh_directory}/swivel.stl" />
-		</geometry>
-		<material name="swivel">
-			<color rgba="0.5 0.5 0.5 1"/>
-		</material>
-	</visual>
-	<collision>
-		<origin xyz="0 0 0" rpy="0 0 0"/>
-		<geometry>
-			<mesh filename="${mesh_directory}/swivel.stl" scale= "1.005 1.005 1.005"/>
-		</geometry>
-	</collision>
-	</link>
-	<gazebo reference="swivel">
-		<material value="Gazebo/Grey"/>
-	</gazebo>
-	<joint name="right_base_swivel_joint" type="continuous">
-		<origin xyz="0 0 -0.04855" rpy="0 0 0"/>
-		<axis xyz="0 0 1"/>
-	    	<!--<joint_properties damping="9.0" />-->
-		<parent link="right_swivel_support"/>
-		<child link="right_swivel"/>
-	</joint>
-<!-- Right swivel Wheel + Hubcap -->
-	<link name="right_swivel_hubcap">
-		<inertial>
-			<mass value="0.01"/>
-			<origin xyz="0 0 0"/>
-			<inertia ixx="0.00012411765597" ixy="0.0" ixz="0.0"
-				 iyy="0.00015218160428" iyz="0.0" izz="0.00011763977943"/>
-  	 	</inertial>
-	<visual name="right_swivel_hubcap">
-		<origin xyz="0 0 0" rpy="0 0 0"/>
-		<geometry name="pioneer_geom">
-			<mesh filename="${mesh_directory}/center_hubcap.stl" />
-		</geometry>
-		<material name="swivel">
-			<color rgba="0.5 0.5 0.5 1"/>
-		</material>
-	</visual>
-	<collision>
-		<origin xyz="0 0 0" rpy="0 0 0"/>
-		<geometry>
-			<mesh filename="${mesh_directory}/center_hubcap.stl" />
-		</geometry>
-	</collision>
-	</link>
-	<gazebo reference="swivel_hubcap">
-		<material value="Gazebo/Grey"/>
-	</gazebo>
-	<joint name="right_swivel_hubcap_joint" type="continuous">
-		<origin xyz="-0.036 0 -0.029" rpy="0 0 0"/>
-		<axis xyz="0 1 0"/>
-		<anchor xyz="0 0 0"/>
-    <joint_properties damping="9.0" />
-	  <parent link="right_swivel"/>
-		<child link="right_swivel_hubcap"/>
-	</joint>
-	<link name="right_swivel_wheel">
-		<inertial>
-			<mass value="2.0"/>
-			<origin xyz="0 0 0"/>
-			<inertia ixx="0.00012411765597" ixy="0.0" ixz="0.0"
-				 iyy="0.00015218160428" iyz="0.0" izz="0.00011763977943"/>
-  	 	</inertial>
-	<visual name="right_swivel_wheel">
-		<origin xyz="0 0 0" rpy="0 0 0"/>
-		<geometry name="swivel_wheel">
-			<mesh filename="${mesh_directory}/center_wheel.stl" />
-		</geometry>
-		<material name="WheelBlack">
-			<color rgba="0.117 0.117 0.117 1"/>
-		</material>
-	</visual>
-	<collision>
-		<origin xyz="0 0 0" rpy=" ${-3.1415927/2} 0 0"/>
-		<geometry>
-			<cylinder radius="0.052" length="0.0422"/>
-		</geometry>
-		      <surface>
-			<friction>
-			  <ode>
-			    <mu>0.8</mu>
-			    <mu2>0.8</mu2>
-			  </ode>
-			</friction>
-		      </surface>
-	</collision>
-	</link>
-	<gazebo reference="swivel_wheel">
-		<material value="Gazebo/Black"/>
-	</gazebo>
-	<joint name="right_swivel_wheel_hubcap_joint" type="fixed">
-		<origin xyz="0 0 0" rpy="0 0 0"/>
-		<parent link="right_swivel_hubcap"/>
-		<child link="right_swivel_wheel"/>
-	</joint>
-  <!-- Left Swivel support-->
-	<link name="left_swivel_support">
-		<inertial>
-			<mass value="0.1"/>
-			<origin xyz="0 0 0" rpy="0 0 0"/>
-			<inertia ixx="0.01" ixy="0" ixz="0"
-				 iyy="0.01" iyz="0" izz="0.01"/>
-  	 	</inertial>
-	<visual name="left_swivel_support_visual">
-		<origin xyz="0 0 0" rpy="0 0 0"/>
-		<geometry name="swivel">
-			<mesh filename="${mesh_directory}/swivel_support.stl" />
-		</geometry>
-		<material name="swivel">
-			<color rgba="0.9 0.9 0.9 1"/>
-		</material>
-	</visual>
-	<collision>
-		<origin xyz="0 0 0" rpy="0 0 0"/>
-		<geometry>
-			<mesh filename="${mesh_directory}/swivel_support.stl" scale= "1.005 1.005 1.005"/>
-		</geometry>
-	</collision>
-	</link>
-	<gazebo reference="swivel">
-		<material value="Gazebo/Grey"/>
-	</gazebo>
-	<joint name="left_base_swivel_support_joint" type="fixed">
-		<origin xyz="-0.215 0.2 -0.0915" rpy="0 0 0"/>
-		<parent link="base_center"/>
-		<child link="left_swivel_support"/>
-	</joint>
-  <!--Left Swivel -->
-	<link name="left_swivel">
-		<inertial>
-			<mass value="2.0"/>
-			<origin xyz="0 0 0" rpy="0 0 0"/>
-			<inertia ixx="0.001" ixy="0" ixz="0"
-				 iyy="0.001" iyz="0" izz="0.001"/>
-  	 	</inertial>
-	<visual name="left_swivel_visual">
-		<origin xyz="0 0 0" rpy="0 0 0"/>
-		<geometry name="swivel">
-			<mesh filename="${mesh_directory}/swivel.stl" />
-		</geometry>
-		<material name="swivel">
-			<color rgba="0.5 0.5 0.5 1"/>
-		</material>
-	</visual>
-	<collision>
-		<origin xyz="0 0 0" rpy="0 0 0"/>
-		<geometry>
-			<mesh filename="${mesh_directory}/swivel.stl"  scale= "1.005 1.005 1.005" />
-		</geometry>
-	</collision>
-	</link>
-	<gazebo reference="swivel">
-		<material value="Gazebo/Grey"/>
-	</gazebo>
-	<joint name="left_base_swivel_joint" type="continuous">
-		<origin xyz="0 0 -0.04855" rpy="0 0 0"/>
-		<axis xyz="0 0 1"/>
-    	<!--<joint_properties damping="9.0" />-->
-		<parent link="left_swivel_support"/>
-		<child link="left_swivel"/>
-	</joint>
-<!-- left swivel Wheel + Hubcap -->
-	<link name="left_swivel_hubcap">
-		<inertial>
-			<mass value="0.01"/>
-			<origin xyz="0 0 0"/>
-			<inertia ixx="0.00012411765597" ixy="0.0" ixz="0.0"
-				 iyy="0.00015218160428" iyz="0.0" izz="0.00011763977943"/>
-  	 	</inertial>
-	<visual name="left_swivel_hubcap">
-		<origin xyz="0 0 0" rpy="0 0 0"/>
-		<geometry name="pioneer_geom">
-			<mesh filename="${mesh_directory}/center_hubcap.stl" />
-		</geometry>
-		<material name="swivel">
-			<color rgba="0.5 0.5 0.5 1"/>
-		</material>
-	</visual>
-	<collision>
-		<origin xyz="0 0 0" rpy="0 0 0"/>
-		<geometry>
-			<mesh filename="${mesh_directory}/center_hubcap.stl" />
-		</geometry>
-	</collision>
-	</link>
-	<gazebo reference="swivel_hubcap">
-		<material value="Gazebo/Grey"/>
-	</gazebo>
-	<joint name="left_swivel_hubcap_joint" type="continuous">
-		<origin xyz="-0.036 0 -0.029" rpy="0 0 0"/>
-		<axis xyz="0 1 0"/>
-		<anchor xyz="0 0 0"/>
-    <joint_properties damping="9.0" />
-	  <parent link="left_swivel"/>
-		<child link="left_swivel_hubcap"/>
-	</joint>
-	<link name="left_swivel_wheel">
-		<inertial>
-			<mass value="2.0"/>
-			<origin xyz="0 0 0"/>
-			<inertia ixx="0.00012411765597" ixy="0.0" ixz="0.0"
-				 iyy="0.00015218160428" iyz="0.0" izz="0.00011763977943"/>
-  	 	</inertial>
-	<visual name="left_swivel_wheel">
-		<origin xyz="0 0 0" rpy="0 0 0"/>
-		<geometry name="swivel_wheel">
-			<mesh filename="${mesh_directory}/center_wheel.stl" />
-		</geometry>
-		<material name="WheelBlack">
-			<color rgba="0.117 0.117 0.117 1"/>
-		</material>
-	</visual>
-	<collision>
-		<origin xyz="0 0 0" rpy=" ${-3.1415927/2} 0 0"/>
-		<geometry>
-			<cylinder radius="0.052" length="0.0422"/>
-		</geometry>
-		      <surface>
-			<friction>
-			  <ode>
-			    <mu>0.8</mu>
-			    <mu2>0.8</mu2>
-			  </ode>
-			</friction>
-		      </surface>
-	</collision>
-	</link>
-	<gazebo reference="right_wheel">
-		<material value="Gazebo/Black"/>
-	</gazebo>
-	<joint name="left_swivel_wheel_hubcap_joint" type="fixed">
-		<origin xyz="0 0 0" rpy="0 0 0"/>
-		<parent link="left_swivel_hubcap"/>
-		<child link="left_swivel_wheel"/>
-	</joint>
-	<!--Left Wheel and hub-->
-	<link name="left_hubcap">
-	     <inertial>
-		<mass value="0.08"/>
-		<origin xyz="0 0 0"/>
-		<inertia ixx="0.012411765597" ixy="0" ixz="0"
-		         iyy="0.015218160428" iyz="0" izz="0.011763977943"/>
-	      </inertial>
-		<visual>
-			<origin xyz="0 0 0" rpy="0 0 0"/>
-			<geometry>
-				<mesh filename="${mesh_directory}/hubcap.stl"/>
-			</geometry>
-			<material name="HubcapWhite">
-				<color rgba="1.0 1.0 1.0 1.0"/>
-			</material>
-		</visual>
-	      <collision>
-		<origin xyz="0 0 0" rpy="0 0 0"/>
-		<geometry>
-		  <mesh filename="${mesh_directory}/hubcap.stl"/>
-		</geometry>
-	      </collision>
-	</link>
-	<joint name="base_left_hub_joint" type="continuous">
-		<origin xyz="0.084 0.35 -0.0835" rpy="0 0 0"/>
-	        <anchor xyz="0 0 0"/>
-	        <joint_properties damping="9.0"  />
-		<parent link="base_center"/>
-		<child link="left_hubcap"/>
-		<axis xyz="0 1 0"/>
-	</joint>
-	<link name="left_wheel">
-	      <inertial>
-		<mass value="15.25"/>
-		<origin xyz="0 0 0"/>
-		<inertia ixx="0.012411765597" ixy="0" ixz="0"
-		         iyy="0.015218160428" iyz="0" izz="0.011763977943"/>
-	      </inertial>
-		<visual>
-			<origin xyz="0 0 0" rpy="0 0 0"/>
-			<geometry>
-				<mesh filename="${mesh_directory}/wheel.stl" />
-			</geometry>
-			<material name="WheelBlack">
-				<color rgba="0.117 0.117 0.117 1"/>
-			</material>
-		</visual>
-	      <collision>
-		<origin xyz="0 0 0" rpy="${-3.1415927/2} 0 0"/>
-		<geometry>
-		  <cylinder radius="0.133" length="0.065"/>
-		</geometry>
-		      <surface>
-			<friction>
-			  <ode>
-			    <mu>0.8</mu>
-			    <mu2>0.8</mu2>
-			  </ode>
-			</friction>
-		      </surface>
-	      </collision>
-	</link>
-	<joint name="left_wheel_joint" type="fixed">
-		<origin xyz="0 0 0" rpy="0 0 0"/>
-		<parent link="left_hubcap"/>
-		<child link="left_wheel"/>
-	</joint>
-	<gazebo reference="left_wheel">
-		<material value="Gazebo/Black"/>
-	</gazebo>
-	<!--Right Wheel and hub-->
-	<link name="right_hubcap">
-	     <inertial>
-		<mass value="0.08"/>
-		<origin xyz="0 0 0"/>
-		<inertia ixx="0.012411765597" ixy="0" ixz="0"
-		         iyy="0.015218160428" iyz="0" izz="0.011763977943"/>
-	      </inertial>
-		<visual>
-			<origin xyz="0 0 0" rpy="0 0 0"/>
-			<geometry>
-				<mesh filename="${mesh_directory}/hubcap.stl"/>
-			</geometry>
-			<material name="HubcapWhite">
-				<color rgba="1.0 1.0 1.0 1.0"/>
-			</material>
-		</visual>
-	      <collision>
-		<origin xyz="0 0 0" rpy="0 0 0"/>
-		<geometry>
-		  <mesh filename="${mesh_directory}/hubcap.stl"/>
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
File: champ_description/urdf/powerbot/powerbot_wheel.xacro (robot description, xacro)
@@ -1,93 +1,81 @@
 <?xml version="1.0"?>
-<robot
-  xmlns:sensor="http://playerstage.sourceforge.net/gazebo/xmlschema/#sensor"
-  xmlns:controller="http://playerstage.sourceforge.net/gazebo/xmlschema/#controller"
-  xmlns:interface="http://playerstage.sourceforge.net/gazebo/xmlschema/#interface"
-  xmlns:xacro="http://ros.org/wiki/xacro"
-  >
+<robot xmlns:xacro="http://ros.org/wiki/xacro">
   <!--<xacro:include filename="$(find p2os_urdf)/defs/materials.xacro"/>-->
   <!-- Properties (Constants) -->
-<xacro:property name="M_PI" value="3.14159"/>
+  <xacro:property name="M_PI" value="3.14159"/>
   <!-- where to find all meshes -->
 <xacro:property name="mesh_directory" value="package://champ_description/meshes/p3dx_meshes"/>
-<!-- Right/Left Hubcap + Wheel -->
-<xacro:macro name="p3dx_wheel" params="suffix parent reflect">
-  <link name="p3dx_${suffix}_wheel">
-    <inertial>
-      <mass value="0.5"/>
-      <origin xyz="0 0 0"/>
-      <inertia ixx="0.012411765597" ixy="0" ixz="0"
-         iyy="0.015218160428" iyz="0" izz="0.011763977943"/>
-      </inertial>
-    <visual name="base_visual">
+  <!-- Right/Left Hubcap + Wheel -->
+  <xacro:macro name="powerbot_wheel" params="suffix parent reflect">
+    <link name="powerbot_${suffix}_wheel">
+      <inertial>
+	<mass value="5.25"/>
+		<origin xyz="0 0 0"/>
+		<inertia ixx="0.012411765597" ixy="0" ixz="0"
+		         iyy="0.015218160428" iyz="0" izz="0.011763977943"/>
+	      </inertial>
+		<visual>
+			<origin xyz="0 0 0" rpy="0 0 0"/>
+			<geometry>
+				<mesh filename="${mesh_directory}/wheel.stl" />
+			</geometry>
+			<material name="WheelBlack">
+				<color rgba="0.117 0.117 0.117 1"/>
+			</material>
+		</visual>
+	<collision>
+		<origin xyz="0 0 0" rpy="${-3.1415927/2} 0 0"/>
+		<geometry>
+		  <cylinder radius="0.133" length="0.065"/>
+		</geometry>
+	</collision>
+    </link>
+    <joint name="base_${suffix}_hubcap_joint" type="fixed">
       <origin xyz="0 0 0" rpy="0 0 0"/>
-      <geometry name="pioneer_geom">
-	<mesh filename="${mesh_directory}/${suffix}_wheel.stl"/>
-      </geometry>
-      <material name="WheelBlack">
-        <color rgba="0.117 0.117 0.117 1"/>
-      </material>
-    </visual>
-    <collision>
-      <origin xyz="0 0 0" rpy="${-3.1415927/2} 0 0"/>
-      <geometry>
-        <!--<mesh filename="package://p2os_urdf/meshes/p3dx_meshes/${suffix}_wheel.stl"/>-->
-        <cylinder radius="0.09" length="0.01"/>
-      </geometry>
-    </collision>
-  </link>
-  <joint name="base_${suffix}_hubcap_joint" type="fixed">
-    <!--<origin xyz="0 ${reflect*0.158} 0.091" rpy="0 0 0"/>-->
-    <origin xyz="0 0 0" rpy="0 0 0"/>
-    <parent link="p3dx_${suffix}_wheel"/>
-    <child link="p3dx_${suffix}_hubcap"/>
-  </joint>
-  <link name="p3dx_${suffix}_hubcap">
-    <inertial>
-      <mass value="0.01"/>
-      <origin xyz="0 0 0"/>
-      <inertia ixx="0.012411765597" ixy="0" ixz="0"
-         iyy="0.015218160428" iyz="0" izz="0.011763977943"/>
-      </inertial>
-  <visual name="base_visual">
-    <origin xyz="0 0 0" rpy="0 0 0"/>
-    <geometry name="pioneer_geom">
-      <mesh filename="${mesh_directory}/${suffix}_hubcap.stl"/>
-    </geometry>
-    <material name="HubcapWhite">
-      <color rgba="1.0 1.0 1.0 1.0"/>
-    </material>
-  </visual>
-  <collision>
-    <origin xyz="0 0 0" rpy="0 0 0"/>
-    <geometry>
-      <box size="0 0 0"/>
-    </geometry>
-  </collision>
-  </link>
-  <transmission type="pr2_mechanism_model/SimpleTransmission" name="${parent}_${suffix}_wheel_trans">
-    <actuator name="base_${suffix}_wheel_motor" />
-    <joint name="base_${suffix}_wheel_joint" />
-    <mechanicalReduction>${reflect * 624/35 * 80/19}</mechanicalReduction>
-  </transmission>
-  <joint name="base_${suffix}_wheel_joint" type="continuous">
-    <axis xyz="0 1 0"/>
-    <anchor xyz="0 0 0"/>
-    <limit effort="100" velocity="100" />
-    <joint_properties damping="0.0" friction="0.0" />
-    <origin xyz="0 ${reflect*0.158} 0.091" rpy="0 0 0"/>
-    <parent link="base_center"/>
-    <child link="p3dx_${suffix}_wheel"/>
-  </joint>
-  <gazebo reference="p3dx_${suffix}_hubcap">
+      <parent link="powerbot_${suffix}_wheel"/>
+      <child link="powerbot_${suffix}_hubcap"/>
+    </joint>
+    <link name="powerbot_${suffix}_hubcap">
+	      <inertial>
+		<mass value="0.08"/>
+		<origin xyz="0 0 0"/>
+		<inertia ixx="0.012411765597" ixy="0" ixz="0"
+		         iyy="0.015218160428" iyz="0" izz="0.011763977943"/>
+	      </inertial>
+		<visual>
+			<origin xyz="0 0 0" rpy="0 0 0"/>
+			<geometry>
+				<mesh filename="${mesh_directory}/hubcap.stl"/>
+			</geometry>
+        <material name="HubcapYellow">
+          <color rgba="1.0 0.811 0.151 1.0"/>
+        </material>
+      </visual>
+    </link>
+    <!-- The transmission tag is used only by ros_control -->
+    <!--<transmission type="pr2_mechanism_model/SimpleTransmission" name="${parent}_${suffix}_wheel_trans">
+        <actuator name="base_${suffix}_wheel_motor" />
+        <joint name="base_${suffix}_wheel_joint" />
+        <mechanicalReduction>${reflect * 624/35 * 80/19}</mechanicalReduction>
+        </transmission>-->
+    <joint name="base_${suffix}_wheel_joint" type="continuous">
+      <axis xyz="0 1 0"/>
+      <anchor xyz="0 0 0"/>
+      <limit effort="100" velocity="100" />
+      <joint_properties damping="0.0" friction="0.0" />
+      <origin xyz="0.084 ${reflect*0.35} -0.0835" rpy="0 0 0"/>
+      <parent link="base_center"/>
+      <child link="powerbot_${suffix}_wheel"/>
+    </joint>
+    <gazebo reference="powerbot_${suffix}_hubcap">
       <material value="Gazebo/Yellow"/>
-  </gazebo>
-  <gazebo reference="p3dx_${suffix}_wheel">
+    </gazebo>
+    <gazebo reference="powerbot_${suffix}_wheel">
       <material value="Gazebo/Black"/>
-      <elem key="mu1" value="0.5" />
-      <elem key="mu2" value="50.0" />
-      <elem key="kp"  value="100000000.0" />
-      <elem key="kd"  value="1.0" />
-  </gazebo>
-</xacro:macro>
+      <mu1>0.5</mu1>
+      <mu2>50.0</mu2>
+      <kp>100000000.0</kp>
+      <kd>1.0</kd>
+    </gazebo>
+  </xacro:macro>
 </robot>
