Commit message: Changed robotNamespace of asus camera plugin to /wam_powerbot. Started fixing robot link collisions (scaled them up by 1.01). Issues: 	- Missing differential drive controller. 	- Fix holy collisions (in progress). 	- Need to spawn urdf in home position. 	- Fix robot tf tree for use with Rviz and Moveit! 	modified:   champ_description/urdf/powerbot/powerbot.xacro 	modified:   champ_description/urdf/sensors/3D_sensor_gazebo.urdf.xacro

File: champ_description/urdf/powerbot/powerbot.xacro (robot description, xacro)
@@ -68,5 +68,5 @@
 			<origin xyz="-0.045 0 ${bcz}" rpy="0 0 0"/>
 			<geometry>
-				<mesh filename="${mesh_directory}/chassis.stl"/>
+				<mesh filename="${mesh_directory}/chassis.stl" scale="1.01 1.01 1.01"/>
 			</geometry>
 		</collision>
@@ -130,5 +130,5 @@
 		<origin xyz="0 0 0" rpy="0 0 0"/>
 		<geometry>
-			<mesh filename="${mesh_directory}/swivel_support.stl" />
+			<mesh filename="${mesh_directory}/swivel_support.stl" scale= "1.005 1.005 1.005"/>
 		</geometry>
 	</collision>
@@ -138,5 +138,5 @@
 	</gazebo>
 	<joint name="right_base_swivel_support_joint" type="fixed">
-		<origin xyz="-0.215 -0.2 -0.091" rpy="0 0 0"/>
+		<origin xyz="-0.215 -0.2 -0.0915" rpy="0 0 0"/>
 		<parent link="base_center"/>
 		<child link="right_swivel_support"/>
@@ -162,5 +162,5 @@
 		<origin xyz="0 0 0" rpy="0 0 0"/>
 		<geometry>
-			<mesh filename="${mesh_directory}/swivel.stl" />
+			<mesh filename="${mesh_directory}/swivel.stl" scale= "1.005 1.005 1.005"/>
 		</geometry>
 	</collision>
@@ -230,5 +230,5 @@
 		<origin xyz="0 0 0" rpy=" ${-3.1415927/2} 0 0"/>
 		<geometry>
-			<cylinder radius="0.0468" length="0.0422"/>
+			<cylinder radius="0.052" length="0.0422"/>
 		</geometry>
 		      <surface>
@@ -270,5 +270,5 @@
 		<origin xyz="0 0 0" rpy="0 0 0"/>
 		<geometry>
-			<mesh filename="${mesh_directory}/swivel_support.stl" />
+			<mesh filename="${mesh_directory}/swivel_support.stl" scale= "1.005 1.005 1.005"/>
 		</geometry>
 	</collision>
@@ -278,5 +278,5 @@
 	</gazebo>
 	<joint name="left_base_swivel_support_joint" type="fixed">
-		<origin xyz="-0.215 0.2 -0.091" rpy="0 0 0"/>
+		<origin xyz="-0.215 0.2 -0.0915" rpy="0 0 0"/>
 		<parent link="base_center"/>
 		<child link="left_swivel_support"/>
@@ -302,5 +302,5 @@
 		<origin xyz="0 0 0" rpy="0 0 0"/>
 		<geometry>
-			<mesh filename="${mesh_directory}/swivel.stl" />
+			<mesh filename="${mesh_directory}/swivel.stl"  scale= "1.005 1.005 1.005" />
 		</geometry>
 	</collision>
@@ -370,5 +370,5 @@
 		<origin xyz="0 0 0" rpy=" ${-3.1415927/2} 0 0"/>
 		<geometry>
-			<cylinder radius="0.0468" length="0.0422"/>
+			<cylinder radius="0.052" length="0.0422"/>
 		</geometry>
 		      <surface>
@@ -441,5 +441,5 @@
 		<origin xyz="0 0 0" rpy="${-3.1415927/2} 0 0"/>
 		<geometry>
-		  <cylinder radius="0.1315" length="0.065"/>
+		  <cylinder radius="0.133" length="0.065"/>
 		</geometry>
 		      <surface>
@@ -512,5 +512,5 @@
 		<origin xyz="0 0 0" rpy="${-3.1415927/2} 0 0"/>
 		<geometry>
-		  <cylinder radius="0.1315" length="0.065"/>
+		  <cylinder radius="0.133" length="0.065"/>
 		</geometry>
 		      <surface>
@@ -601,6 +601,6 @@
     <updateRate>100.0</updateRate>
     <robotNamespace>/</robotNamespace>
-    <leftJoint>base_right_wheel_joint</leftJoint>
-    <rightJoint>base_left_wheel_joint</rightJoint>
+    <leftJoint>left_hub_joint</leftJoint>
+    <rightJoint>right_hub_joint</rightJoint>
     <wheelSeparation>0.39</wheelSeparation>
     <wheelDiameter>0.15</wheelDiameter>

File: champ_description/urdf/sensors/3D_sensor_gazebo.urdf.xacro (robot description, xacro)
@@ -20,4 +20,5 @@
         </camera>
         <plugin name="kinect_camera_controller" filename="libgazebo_ros_openni_kinect.so">
+	<robotNamespace>/wam_powerbot</robotNamespace>
           <cameraName>camera</cameraName>
           <alwaysOn>true</alwaysOn>

Commit message: Working differential drive controller.
Issues:
            - Powerbot refuses to be stationary.
		- Suspects: inertial tensor matrices, swivel wheels, joint friction?
            - Fix holy collisions (in progress).
            - Need to spawn urdf in home position.
            - Fix robot tf tree for use with Rviz and Moveit!

File: champ_description/urdf/powerbot/powerbot.xacro (robot description, xacro)
@@ -172,5 +172,5 @@
 		<origin xyz="0 0 -0.04855" rpy="0 0 0"/>
 		<axis xyz="0 0 1"/>
-	    	<joint_properties damping="9.0" />
+	    	<!--<joint_properties damping="9.0" />-->
 		<parent link="right_swivel_support"/>
 		<child link="right_swivel"/>
@@ -312,5 +312,5 @@
 		<origin xyz="0 0 -0.04855" rpy="0 0 0"/>
 		<axis xyz="0 0 1"/>
-    	<joint_properties damping="9.0" />
+    	<!--<joint_properties damping="9.0" />-->
 		<parent link="left_swivel_support"/>
 		<child link="left_swivel"/>
@@ -414,5 +414,5 @@
 	      </collision>
 	</link>
-	<joint name="left_hub_joint" type="continuous">
+	<joint name="base_left_hub_joint" type="continuous">
 		<origin xyz="0.084 0.35 -0.0835" rpy="0 0 0"/>
 	        <anchor xyz="0 0 0"/>
@@ -424,5 +424,5 @@
 	<link name="left_wheel">
 	      <inertial>
-		<mass value="5.25"/>
+		<mass value="15.25"/>
 		<origin xyz="0 0 0"/>
 		<inertia ixx="0.012411765597" ixy="0" ixz="0"
@@ -485,5 +485,5 @@
 	      </collision>
 	</link>
-	<joint name="right_hub_joint" type="continuous">
+	<joint name="base_right_hub_joint" type="continuous">
 		<origin xyz="0.084 -0.35 -0.0835" rpy="0 0 0"/>
 	        <anchor xyz="0 0 0"/>
@@ -495,5 +495,5 @@
 	<link name="right_wheel">
 	      <inertial>
-		<mass value="5.25"/>
+		<mass value="15.25"/>
 		<origin xyz="0 0 0"/>
 		<inertia ixx="0.012411765597" ixy="0" ixz="0"
@@ -597,18 +597,39 @@
  -->
 <!--Actually include  "skid_steer_drive_controller" in robot urdf-->
-<p3at_gazebo_ext/>
-<xacro:macro name="p3at_gazebo_ext">
-<gazebo>
-  <plugin name="skid_steer_drive_controller" filename="libgazebo_ros_skid_steer_drive.so">
-    <updateRate>100.0</updateRate>
-    <leftJoint>left_hub_joint</leftJoint>
-    <rightJoint>right_hub_joint</rightJoint>
-    <wheelSeparation>0.39</wheelSeparation>
-    <wheelDiameter>0.26</wheelDiameter>
-    <robotBaseFrame>base_center</robotBaseFrame>
-    <torque>200</torque>
-    <topicName>cmd_vel</topicName>
-  </plugin>
-</gazebo>
-</xacro:macro>
+  <gazebo>
+    <!-- Robot locomotion plugin -->
+	<plugin name="differential_drive_controller" filename="libgazebo_ros_diff_drive.so">
+      <legacyMode>false</legacyMode>
+      <alwaysOn>true</alwaysOn>
+	  <updateRate>100.0</updateRate>
+	  <leftJoint>base_left_hub_joint</leftJoint>
+      <rightJoint>base_right_hub_joint</rightJoint>
+	  <wheelSeparation>0.42</wheelSeparation>
+	  <wheelDiameter>0.263</wheelDiameter>
+	  <wheelTorque>5</wheelTorque>
+      <wheelAcceleration>0</wheelAcceleration>
+      <robotNamespace>wam_powerbot</robotNamespace>
+	  <commandTopic>cmd_vel</commandTopic>
+	  <odometryTopic>odom</odometryTopic>
+      <odometrySource>world</odometrySource><!--Other option is Encoder-->
+	  <odometryFrame>odom</odometryFrame>
+      <robotBaseFrame>base_center</robotBaseFrame>
+      <publishTf>1</publishTf>
+      <publishWheelTF>false</publishWheelTF>
+      <publishWheelJointState>false</publishWheelJointState>
+      <rosDebugLevel>Warn</rosDebugLevel>
+	</plugin>
+    <!-- Fake localization plugin -->
+    <plugin name="ground_truth_odometry" filename="libgazebo_ros_p3d.so">
+	  <alwaysOn>true</alwaysOn>
+	  <updateRate>100.0</updateRate>
+	  <bodyName>base_center</bodyName>
+	  <topicName>base_pose_ground_truth</topicName>
+	  <gaussianNoise>0.01</gaussianNoise>
+	  <frameName>world</frameName><!--other option is World-->
+      <!-- initialize odometry for fake localization-->
+	  <xyzOffsets>0 0 0</xyzOffsets>
+	  <rpyOffsets>0 0 0</rpyOffsets>
+	</plugin>
+  </gazebo>
 </robot>

Commit message: Successfully added ball swivels. Base is able to remain relatively stationary. Issues: 	- Base cannot drive straight (does donuts around left front wheel). 		- Surface contact point with the ground keeps disappearing. 	- WAM hand and base collisions not detected. 		- Try to inflate collision meshes for WAM links.

File: champ_description/urdf/powerbot/powerbot.xacro (robot description, xacro)
@@ -16,5 +16,5 @@
   <xacro:include filename="$(find champ_description)/urdf/powerbot/powerbot_wheel.xacro"/>
   <!-- Include powerbot swivel wheels -->
-  <xacro:include filename="$(find champ_description)/urdf/powerbot/powerbot_swivel_wheel.xacro"/>
+  <xacro:include filename="$(find champ_description)/urdf/powerbot/powerbot_swivel_ball.xacro"/>
   <!-- where to find all meshes -->
   <xacro:property name="mesh_directory" value="package://champ_description/meshes/p3dx_meshes"/>
@@ -112,6 +112,6 @@
 		<material value="Gazebo/Black"/>
 	</gazebo>
- <xacro:powerbot_swivel_wheel suffix="left" parent="base_center" reflect="1"/>
-  <xacro:powerbot_swivel_wheel suffix="right" parent="base_center" reflect="-1"/>
+ <xacro:powerbot_swivel_ball suffix="left" parent="base_center" reflect="1"/>
+  <xacro:powerbot_swivel_ball suffix="right" parent="base_center" reflect="-1"/>
   <xacro:powerbot_wheel suffix="left" parent="base_center" reflect="1"/>
   <xacro:powerbot_wheel suffix="right" parent="base_center" reflect="-1"/>

File: champ_description/urdf/powerbot/powerbot_wheel.xacro (robot description, xacro)
@@ -28,5 +28,8 @@
 		<geometry>
 		  <cylinder radius="0.133" length="0.065"/>
-		</geometry>
+		</geometry><!--
+			<geometry>
+				<mesh filename="${mesh_directory}/wheel.stl" scale= "1.005 1.005 1.005"/>
+			</geometry>-->
 	</collision>
     </link>

Commit message: Added ball joints to ball swivels (used three continuous joints at the same origin) Issues:         - Base still drifts                 - Surface contact point with the ground keeps disappearing.         - WAM hand and base collisions not detected.                 - Try to inflate collision meshes for WAM links 	- unable to visualise color for base

File: champ_description/urdf/powerbot/powerbot.xacro (robot description, xacro)
@@ -63,7 +63,4 @@
 				<mesh filename="${mesh_directory}/chassis.stl"/>
 			</geometry>
-	<material name="ChassisRed">
-		<color rgba="0.8 0.0 0.0 1.0"/>
-	</material>
 		</visual>
 		<collision>
@@ -75,5 +72,5 @@
 	</link>
 	<gazebo reference="base_center">
-		 <material>Gazebo/Red</material>
+		 <material>Gazebo/Yellow</material>
 	</gazebo>
 <!-- Top -->

File: champ_description/urdf/powerbot/powerbot_swivel_ball.xacro (robot description, xacro)
@@ -76,34 +76,56 @@
 		<material value="Gazebo/Grey"/>
 	</gazebo>
-<!-- ${suffix} support swivel ball joint-->
-<joint name="${suffix}_ballRoot_joint" type="continuous" >
+<!-- ${suffix} support swivel ball joint -->
+<joint name="${suffix}_ballRoot_joint" type="fixed" >
     <origin xyz="0 0 0" />
     <parent link="powerbot_${suffix}_swivel_support" />
-    <child link="powerbot_${suffix}_swivel_ball" />
-    <axis xyz="1 1 1" />
-    <dynamics damping="0.005" />
+    <child link="${suffix}_ball" />
 </joint>
-<!--
-<link name="${suffix}_ball" />
+<link name="${suffix}_ball" >
+<inertial>
+	<mass value="2.0"/>
+	<origin xyz="0 0 0"/>
+	<inertia ixx="0.00288" ixy="0.0" ixz="0.0"
+		 iyy="0.00288" iyz="0.0" izz="0.00288"/>
+</inertial>
+  </link>
 <joint name="${suffix}_ballPsi_joint" type="continuous" >
+    <origin xyz="0 0 0" rpy="0 0 0"/>
     <parent link="${suffix}_ball" />
     <child link="${suffix}_ball_psi_link" />
     <axis xyz="0 0 1" />
-    <dynamics damping="0.005" />
+    <dynamics damping="0.09" />
 </joint>
-<link name="${suffix}_ball_psi_link" />
+<link name="${suffix}_ball_psi_link" >
+<inertial>
+	<mass value="2.0"/>
+	<origin xyz="0 0 0"/>
+	<inertia ixx="0.00288" ixy="0.0" ixz="0.0"
+		 iyy="0.00288" iyz="0.0" izz="0.00288"/>
+</inertial>
+  </link>
 <joint name="${suffix}_ballTheta_joint" type="continuous" >
+    <origin xyz="0 0 0" rpy="0 0 0"/>
     <parent link="${suffix}_ball_psi_link"/>
     <child link="${suffix}_ball_theta_link"/>
     <axis xyz="0 1 0" />
-    <dynamics damping="0.005" />
+    <dynamics damping="0.09" />
 </joint>
-<link name="${suffix}_ball_theta_link" />
+<link name="${suffix}_ball_theta_link" >
+	<inertial>
+		<mass value="2.0"/>
+		<origin xyz="0 0 0"/>
+		<inertia ixx="0.00288" ixy="0.0" ixz="0.0"
+			 iyy="0.00288" iyz="0.0" izz="0.00288"/>
+	</inertial>
+  </link>
 <joint name="${suffix}_ballPhi_joint" type="continuous" >
+    <origin xyz="0 0 0" rpy="0 0 0"/>
     <parent link="${suffix}_ball_theta_link"/>
     <child link="powerbot_${suffix}_swivel_ball"/>
     <axis xyz="1 0 0" />
-    <dynamics damping="0.005" />
+    <dynamics damping="0.09" />
 </joint>
+<!--
 -->
  <!-- Swivel ball -->
@@ -133,6 +155,6 @@
     <gazebo reference="powerbot_${suffix}_swivel_ball">
       <material value="Gazebo/Grey"/>
-      <mu1>0.5</mu1>
-      <mu2>50.0</mu2>
+      <mu1>100</mu1>
+      <mu2>200</mu2>
       <kp>100000000.0</kp>
       <kd>1.0</kd>

File: champ_description/urdf/powerbot/powerbot_wheel.xacro (robot description, xacro)
@@ -67,10 +67,10 @@
       <limit effort="100" velocity="100" />
       <joint_properties damping="0.0" friction="0.0" />
-      <origin xyz="0.084 ${reflect*0.35} -0.0835" rpy="0 0 0"/>
+      <origin xyz="0.084 ${reflect*0.35} -0.07" rpy="0 0 0"/>
       <parent link="base_center"/>
       <child link="powerbot_${suffix}_wheel"/>
     </joint>
     <gazebo reference="powerbot_${suffix}_hubcap">
-      <material value="Gazebo/Yellow"/>
+      <material value="Gazebo/White"/>
     </gazebo>
     <gazebo reference="powerbot_${suffix}_wheel">

Commit message: Removed base wheels to stop drifting problem. Issues: 	- WAM collision meshes have holes. 	- WAM joint PID parameters still untuned. 	- Rviz does not visualise joint states topic (Mismatching msg types?).

File: champ_description/urdf/powerbot/powerbot.xacro (robot description, xacro)
@@ -5,7 +5,8 @@
 	xmlns:interface="http://playerstage.sourceforge.net/gazebo/xmlschema/#interface"
 	xmlns:xacro="http://ros.org/wiki/xacro">
- <!-- robot name -->
+<xacro:macro name="powerbot"/>
+ <!-- robot name
   <xacro:macro name="powerbot" params="prefix parent_link xyz rpy">
-    <joint name ="${prefix}/world_joint" type="planar">
+    <joint name ="${prefix}/world_joint" type="fixed">
       <parent link="${parent_link}"/>
       <child link="base_center"/>
@@ -13,4 +14,5 @@
     </joint>
   </xacro:macro>
+ -->
   <!-- Include powerbot wheels -->
   <xacro:include filename="$(find champ_description)/urdf/powerbot/powerbot_wheel.xacro"/>
@@ -54,7 +56,7 @@
 	  <mass value="120.0"/>
 	  <origin xyz="-0.045 0 ${bcz}"/>
-	  <inertia ixx="0.4255" ixy="0.0"    ixz="0.0"
-		   		iyy="0.4955" iyz="0.0"
-	          			     izz="0.7441"/>
+	  <inertia ixx="1" ixy="0.0"    ixz="0.0"
+		   		iyy="1" iyz="0.0"
+	          			     izz="1"/>
 	</inertial>
 		<visual name="base_visual">
@@ -73,4 +75,5 @@
 	<gazebo reference="base_center">
 		 <material>Gazebo/Yellow</material>
+    		<static>true</static>
 	</gazebo>
 <!-- Top -->
@@ -109,8 +112,10 @@
 		<material value="Gazebo/Black"/>
 	</gazebo>
+  <!--
  <xacro:powerbot_swivel_ball suffix="left" parent="base_center" reflect="1"/>
   <xacro:powerbot_swivel_ball suffix="right" parent="base_center" reflect="-1"/>
   <xacro:powerbot_wheel suffix="left" parent="base_center" reflect="1"/>
   <xacro:powerbot_wheel suffix="right" parent="base_center" reflect="-1"/>
+-->
 <!-- Front + Back Sonar
 	<link name="front_sonar">

File: champ_description/urdf/wam_powerbot.xacro (robot description, xacro)
@@ -26,6 +26,7 @@
   </xacro:asus_camera_model>
   -->
-<!-- Root link is in the world frame-->
+<!-- Root link is in the world frame
 <link name="world"/>
+-->
 <!-- ArmStuff -->
 <!-- BHand -->
@@ -33,5 +34,5 @@
 <!-- 7-DOF Wam on top of top plate-->
 <xacro:wam_7dof prefix="wam" parent_link="arm_plate" xyz="0.22 0.0 0.05" rpy="0 0 0" />
-<xacro:powerbot prefix="powerbot" parent_link="world" xyz="0.0 0.0 0.0" rpy="0 0 0" />
+<xacro:powerbot/>
 <!--Joint Controllers
 - ARM

Commit message: Added cricket world launch file for throwing task.

File: champ_description/urdf/powerbot/powerbot.xacro (robot description, xacro)
@@ -39,10 +39,10 @@
 		</material>
 	</visual>
-	<collision>
+	<!--<collision>
 		<origin xyz="0.2 0 0.03" rpy="0 0 0"/>
 		<geometry>
 			<box size="0.45 0.75 0.05"/>
 		</geometry>
-	</collision>
+	</collision>-->
 </link>
 <joint name="arm_plate_joint" type="fixed">
@@ -66,10 +66,10 @@
 			</geometry>
 		</visual>
-		<collision>
+		<!--<collision>
 			<origin xyz="-0.045 0 ${bcz}" rpy="0 0 0"/>
 			<geometry>
 				<mesh filename="${mesh_directory}/chassis.stl" scale="1.01 1.01 1.01"/>
 			</geometry>
-		</collision>
+		</collision>-->
 	</link>
 	<gazebo reference="base_center">
@@ -102,10 +102,10 @@
 			</material>
 		</visual>
-		<collision>
+		<!--<collision>
 			<origin xyz="0 0 0" rpy="0 0 0"/>
 			<geometry>
 				<mesh filename="${mesh_directory}/top.stl" />
 			</geometry>
-		</collision>
+		</collision>-->
 	</link>
 	<gazebo reference="top_plate">
