Commit message: - Moved WAM joint jontroller definitions from wam_powerbot.xacro to wam7_bball.urdf.xacro    and wam7_bhand.urdf.xacro.  - Moved all unrelated xacro files into .../urdf/wam/defs  - Added eef (end effector type) and control (controller type) args to champ_world.launch 	- Created controller launch files for each eef and control arg combination.  - Deleted redundant files  - Fixed visualisation in Rviz visualisation (was a TF tree issue ).
 Issues:
        - WAM collision meshes have holes.
        - WAM joint PID parameters still untuned.
	- Still need to fix inertias and surface friction for base wheels (currently disabled).

	modified:   champ_description/launch/champ_world.launch
	modified:   champ_description/launch/wam_bball.launch
	modified:   champ_description/launch/wam_bhand.launch
	deleted:    champ_description/urdf/box_wam_powerbot.urdf
	new file:   champ_description/urdf/champ_bball.xacro
	new file:   champ_description/urdf/champ_bhand.xacro
	renamed:    champ_description/urdf/wam/arm.urdf.xacro -> champ_description/urdf/wam/defs/arm.urdf.xacro
	renamed:    champ_description/urdf/wam/ball.urdf.xacro -> champ_description/urdf/wam/defs/ball.urdf.xacro
	renamed:    champ_description/urdf/wam/barrett.urdf.xacro -> champ_description/urdf/wam/defs/barrett.urdf.xacro
	renamed:    champ_description/urdf/wam/common.urdf.xacro -> champ_description/urdf/wam/defs/common.urdf.xacro
	renamed:    champ_description/urdf/wam/components.urdf.xacro -> champ_description/urdf/wam/defs/components.urdf.xacro
	renamed:    champ_description/urdf/wam/hand.urdf.xacro -> champ_description/urdf/wam/defs/hand.urdf.xacro
	renamed:    champ_description/urdf/wam/wam4.urdf.xacro -> champ_description/urdf/wam/defs/wam4.urdf.xacro
	renamed:    champ_description/urdf/wam/wam4_stump.urdf.xacro -> champ_description/urdf/wam/defs/wam4_stump.urdf.xacro
	renamed:    champ_description/urdf/wam/wam7.urdf.xacro -> champ_description/urdf/wam/defs/wam7.urdf.xacro
	renamed:    champ_description/urdf/wam/wam_4dof_wam_bhand.urdf.xacro -> champ_description/urdf/wam/defs/wam_4dof_wam_bhand.urdf.xacro
	renamed:    champ_description/urdf/wam/wam_top.urdf.xacro -> champ_description/urdf/wam/defs/wam_top.urdf.xacro
	renamed:    champ_description/urdf/wam_ball_powerbot.xacro -> champ_description/urdf/wam/wam7_bball.urdf.xacro
	renamed:    champ_description/urdf/wam_ball.xacro -> champ_description/urdf/wam/wam7_bball.xacro
	renamed:    champ_description/urdf/wam_bhand_powerbot.xacro -> champ_description/urdf/wam/wam7_bhand.urdf.xacro
	renamed:    champ_description/urdf/wam_powerbot.xacro -> champ_description/urdf/wam/wam7_bhand.xacro
	deleted:    champ_description/urdf/wam/wam_7dof_wam_bhand.urdf.xacro
	modified:   champ_description/urdf/wam/wam_bhand.urdf
	deleted:    champ_description/urdf/wam_box.urdf
	deleted:    champ_description/urdf/wam_box.xacro
	deleted:    champ_description/urdf/wam_powerbot.urdf
	new file:   wam_control/launch/wam_bball_effort_control.launch
	new file:   wam_control/launch/wam_bball_position_control.launch
	renamed:    wam_control/launch/wam_control_effort.launch -> wam_control/launch/wam_bhand_effort_control.launch
	renamed:    wam_control/launch/wam_control_position.launch -> wam_control/launch/wam_bhand_position_control.launch

File: champ_description/urdf/wam/wam7_bhand.urdf.xacro (robot description, xacro)
@@ -3,5 +3,5 @@
   xmlns:xacro="http://www.ros.org/wiki/xacro">
   <!-- Includea all the WAM stuff -->
-  <xacro:include filename="$(find champ_description)/urdf/wam/wam_top.urdf.xacro"/>
+  <xacro:include filename="$(find champ_description)/urdf/wam/defs/wam_top.urdf.xacro"/>
   <!-- Root link is in the world frame-->
   <link name="world"/>
@@ -10,4 +10,184 @@
   <!-- BHand -->
   <xacro:bhand prefix="wam/bhand" parent_link="wam/wrist_palm_link" xyz="0 0 0.06" rpy="0 0 1.57079"/>
-  <!-- WAM joint Controllers -->
+  <!-- ARM Joint Controllers
+      - wam/base_yaw_joint
+      - wam/shoulder_pitch_joint
+      - wam/shoulder_yaw_joint
+      - wam/elbow_pitch_joint
+      - wam/wrist_yaw_joint
+      - wam/wrist_pitch_joint
+      - wam/palm_yaw_joint
+-->
+<!-- wam/base_yaw_joint -->
+  <transmission name="w1">
+    <type>transmission_interface/SimpleTransmission</type>
+    <joint name="wam/base_yaw_joint">
+      <hardwareInterface>hardware_interface/EffortJointInterface</hardwareInterface>
+    </joint>
+    <actuator name="motor1">
+      <hardwareInterface>hardware_interface/EffortJointInterface</hardwareInterface>
+      <mechanicalReduction>1</mechanicalReduction>
+    </actuator>
+  </transmission>
+<!-- wam/shoulder_pitch_joint -->
+  <transmission name="w2">
+    <type>transmission_interface/SimpleTransmission</type>
+    <joint name="wam/shoulder_pitch_joint">
+      <hardwareInterface>hardware_interface/EffortJointInterface</hardwareInterface>
+    </joint>
+    <actuator name="motor2">
+      <hardwareInterface>hardware_interface/EffortJointInterface</hardwareInterface>
+      <mechanicalReduction>1</mechanicalReduction>
+    </actuator>
+  </transmission>
+<!-- wam/shoulder_yaw_joint -->
+  <transmission name="w3">
+    <type>transmission_interface/SimpleTransmission</type>
+    <joint name="wam/shoulder_yaw_joint">
+      <hardwareInterface>hardware_interface/EffortJointInterface</hardwareInterface>
+    </joint>
+    <actuator name="motor3">
+      <hardwareInterface>hardware_interface/EffortJointInterface</hardwareInterface>
+      <mechanicalReduction>1</mechanicalReduction>
+    </actuator>
+  </transmission>
+<!-- wam/elbow_pitch_joint -->
+  <transmission name="w4">
+    <type>transmission_interface/SimpleTransmission</type>
+    <joint name="wam/elbow_pitch_joint">
+      <hardwareInterface>hardware_interface/EffortJointInterface</hardwareInterface>
+    </joint>
+    <actuator name="motor4">
+      <hardwareInterface>hardware_interface/EffortJointInterface</hardwareInterface>
+      <mechanicalReduction>1</mechanicalReduction>
+    </actuator>
+  </transmission>
+<!-- wam/wrist_yaw_joint -->
+  <transmission name="w5">
+    <type>transmission_interface/SimpleTransmission</type>
+    <joint name="wam/wrist_yaw_joint">
+      <hardwareInterface>hardware_interface/EffortJointInterface</hardwareInterface>
+    </joint>
+    <actuator name="motor5">
+      <hardwareInterface>hardware_interface/EffortJointInterface</hardwareInterface>
+      <mechanicalReduction>1</mechanicalReduction>
+    </actuator>
+  </transmission>
+<!-- wam/wrist_pitch_joint -->
+  <transmission name="w6">
+    <type>transmission_interface/SimpleTransmission</type>
+    <joint name="wam/wrist_pitch_joint">
+      <hardwareInterface>hardware_interface/EffortJointInterface</hardwareInterface>
+    </joint>
+    <actuator name="motor6">
+      <hardwareInterface>hardware_interface/EffortJointInterface</hardwareInterface>
+      <mechanicalReduction>1</mechanicalReduction>
+    </actuator>
+  </transmission>
+<!-- wam/palm_yaw_joint -->
+  <transmission name="w7">
+    <type>transmission_interface/SimpleTransmission</type>
+    <joint name="wam/palm_yaw_joint">
+      <hardwareInterface>hardware_interface/EffortJointInterface</hardwareInterface>
+    </joint>
+    <actuator name="motor7">
+      <hardwareInterface>hardware_interface/EffortJointInterface</hardwareInterface>
+      <mechanicalReduction>1</mechanicalReduction>
+    </actuator>
+  </transmission>
+<!-- BHAND Joint Controllers
+      - wam/bhand/finger_1/med_joint
+      - wam/bhand/finger_1/dist_joint
+      - wam/bhand/finger_2/med_joint
+      - wam/bhand/finger_2/dist_joint
+      - wam/bhand/finger_3/dist_joint
+-->
+<!-- wam/bhand/finger_1/prox_joint -->
+  <transmission name="f1_prox">
+    <type>transmission_interface/SimpleTransmission</type>
+    <joint name="wam/bhand/finger_1/prox_joint">
+      <hardwareInterface>hardware_interface/EffortJointInterface</hardwareInterface>
+    </joint>
+    <actuator name="motor8_1">
+      <hardwareInterface>hardware_interface/EffortJointInterface</hardwareInterface>
+      <mechanicalReduction>1</mechanicalReduction>
+    </actuator>
+  </transmission>
+<!-- wam/bhand/finger_1/med_joint -->
+  <transmission name="f1_med">
+    <type>transmission_interface/SimpleTransmission</type>
+    <joint name="wam/bhand/finger_1/med_joint">
+      <hardwareInterface>hardware_interface/EffortJointInterface</hardwareInterface>
+    </joint>
+    <actuator name="motor8_2">
+      <hardwareInterface>hardware_interface/EffortJointInterface</hardwareInterface>
+      <mechanicalReduction>1</mechanicalReduction>
+    </actuator>
+  </transmission>
+<!-- wam/bhand/finger_1/dist_joint -->
+  <transmission name="f1_dist">
+    <type>transmission_interface/SimpleTransmission</type>
+    <joint name="wam/bhand/finger_1/dist_joint">
+      <hardwareInterface>hardware_interface/EffortJointInterface</hardwareInterface>
+    </joint>
+    <actuator name="motor8_3">
+      <hardwareInterface>hardware_interface/EffortJointInterface</hardwareInterface>
+      <mechanicalReduction>1</mechanicalReduction>
+    </actuator>
+  </transmission>
+<!-- wam/bhand/finger_2/prox_joint -->
+  <transmission name="f2_prox">
+    <type>transmission_interface/SimpleTransmission</type>
+    <joint name="wam/bhand/finger_2/prox_joint">
+      <hardwareInterface>hardware_interface/EffortJointInterface</hardwareInterface>
+    </joint>
+    <actuator name="motor9_1">
+      <hardwareInterface>hardware_interface/EffortJointInterface</hardwareInterface>
+      <mechanicalReduction>1</mechanicalReduction>
+    </actuator>
+  </transmission>
+<!-- wam/bhand/finger_2/med_joint -->
+  <transmission name="f2_med">
+    <type>transmission_interface/SimpleTransmission</type>
+    <joint name="wam/bhand/finger_2/med_joint">
+      <hardwareInterface>hardware_interface/EffortJointInterface</hardwareInterface>
+    </joint>
+    <actuator name="motor9_2">
+      <hardwareInterface>hardware_interface/EffortJointInterface</hardwareInterface>
+      <mechanicalReduction>1</mechanicalReduction>
+    </actuator>
+  </transmission>
+<!-- wam/bhand/finger_2/dist_joint -->
+  <transmission name="f2_dist">
+    <type>transmission_interface/SimpleTransmission</type>
+    <joint name="wam/bhand/finger_2/dist_joint">
+      <hardwareInterface>hardware_interface/EffortJointInterface</hardwareInterface>
+    </joint>
+    <actuator name="motor9_3">
+      <hardwareInterface>hardware_interface/EffortJointInterface</hardwareInterface>
+      <mechanicalReduction>1</mechanicalReduction>
+    </actuator>
+  </transmission>
+<!-- wam/bhand/finger_3/med_joint -->
+  <transmission name="f3_med">
+    <type>transmission_interface/SimpleTransmission</type>
+    <joint name="wam/bhand/finger_3/med_joint">
+      <hardwareInterface>hardware_interface/EffortJointInterface</hardwareInterface>
+    </joint>
+    <actuator name="motor10_1">
+      <hardwareInterface>hardware_interface/EffortJointInterface</hardwareInterface>
+      <mechanicalReduction>1</mechanicalReduction>
+    </actuator>
+  </transmission>
+<!-- wam/bhand/finger_3/dist_joint -->
+  <transmission name="f3_dist">
+    <type>transmission_interface/SimpleTransmission</type>
+    <joint name="wam/bhand/finger_3/dist_joint">
+      <hardwareInterface>hardware_interface/EffortJointInterface</hardwareInterface>
+    </joint>
+    <actuator name="motor10_2">
+      <hardwareInterface>hardware_interface/EffortJointInterface</hardwareInterface>
+      <mechanicalReduction>1</mechanicalReduction>
+    </actuator>
+  </transmission>
 </robot>

File: champ_description/urdf/wam/wam7_bhand.xacro (robot description, xacro)
@@ -1,47 +1,12 @@
 <?xml version="1.0"?>
-<robot name="wam_powerbot"
-	xmlns:sensor="http://playerstage.sourceforge.net/gazebo/xmlschema/#sensor"
-	xmlns:controller="http://playerstage.sourceforge.net/gazebo/xmlschema/#controller"
-	xmlns:interface="http://playerstage.sourceforge.net/gazebo/xmlschema/#interface"
-	xmlns:xacro="http://ros.org/wiki/xacro">
+<robot xmlns:xacro="http://www.ros.org/wiki/xacro">
   <!-- Includea all the WAM stuff -->
-  <xacro:include filename="$(find champ_description)/urdf/wam/wam_top.urdf.xacro"/>
-<link name="cam"/>
-  <!-- Include powerbot -->
- <xacro:include filename="$(find champ_description)/urdf/powerbot/powerbot.xacro"/>
-<!-- Load kinect from turtlebot_description and position it at origin from asus_cal -->
-<xacro:include filename="$(find champ_description)/urdf/sensors/asus/asus_cal.xacro"/>
-<xacro:include filename="$(find champ_description)/urdf/sensors/asus/asus_xtion_pro.urdf.xacro"/>
-<xacro:sensor_asus_xtion_pro parent="cam"/>
-<joint name="cam_joint" type="fixed">
-	<origin xyz="${asus_x} ${asus_y} ${asus_z}" rpy="${asus_roll} ${asus_pitch} ${asus_yaw}"/>
-	<parent link="base_center"/>
-	<child link="cam"/>
-</joint>
-<!-- Kinect stuff
-  <xacro:include filename="$(find champ_description)/urdf/asus/asus.xacro"/>
-  <xacro:include filename="$(find champ_description)/urdf/asus/asus_cal.xacro"/>
-  <xacro:asus_camera_model name="kinect" parent="base_center">
-       <origin xyz="${asus_x} ${asus_y} ${asus_z}" rpy="${asus_roll} ${asus_pitch} ${asus_yaw}"/>
-  </xacro:asus_camera_model>
-  -->
-<!-- Root link is in the world frame-->
-<link name="world"/>
-<joint name="world_fixed_joint" type="fixed">
-<origin xyz="0 0 0" rpy="0 0 0"/>
-<parent link="world"/>
-<child link="base_center"/>
-</joint>
-<!-- ArmStuff -->
-<!-- BHand
-<xacro:bhand prefix="wam/bhand" parent_link="wam/wrist_palm_link" xyz="0 0 0.06" rpy="0 0 0"/>
--->
-<!--Ball-->
-<xacro:bball parent_link="wam/wrist_palm_link" prefix="wam/ball" xyz="0 0 0.06" rpy="0 0 0"/>
-<!-- 7-DOF Wam on top of top plate-->
-<xacro:wam_7dof prefix="wam" parent_link="arm_plate" xyz="0.22 0.0 0.05" rpy="0 0 0" />
-<xacro:powerbot/>
-<!--Joint Controllers
-- ARM
+  <xacro:include filename="$(find champ_description)/urdf/wam/defs/wam_top.urdf.xacro"/>
+<xacro:macro name="wam7_bhand" params="prefix parent xyz rpy">
+  <!-- 7-DOF Wam -->
+  <xacro:wam_7dof prefix="${prefix}" parent_link="${parent}" xyz="${xyz}" rpy="${rpy}" />
+  <!-- BHand -->
+  <xacro:bhand prefix="${prefix}/bhand" parent_link="${prefix}/wrist_palm_link" xyz="0 0 0.06" rpy="0 0 1.57079"/>
+  <!-- ARM Joint Controllers
       - wam/base_yaw_joint
       - wam/shoulder_pitch_joint
@@ -51,10 +16,4 @@
       - wam/wrist_pitch_joint
       - wam/palm_yaw_joint
-- HAND
-      - wam/bhand/finger_1/med_joint
-      - wam/bhand/finger_1/dist_joint
-      - wam/bhand/finger_2/med_joint
-      - wam/bhand/finger_2/dist_joint
-      - wam/bhand/finger_3/dist_joint
 -->
 <!-- wam/base_yaw_joint -->
@@ -135,4 +94,11 @@
     </actuator>
   </transmission>
+<!-- BHAND Joint Controllers
+      - wam/bhand/finger_1/med_joint
+      - wam/bhand/finger_1/dist_joint
+      - wam/bhand/finger_2/med_joint
+      - wam/bhand/finger_2/dist_joint
+      - wam/bhand/finger_3/dist_joint
+-->
 <!-- wam/bhand/finger_1/prox_joint -->
   <transmission name="f1_prox">
@@ -223,8 +189,4 @@
     </actuator>
   </transmission>
-<gazebo>
-  <plugin name="gazebo_ros_control" filename="libgazebo_ros_control.so">
-    <robotNamespace>/wam_powerbot</robotNamespace>
-  </plugin>
-</gazebo>
+</xacro:macro>
 </robot>
