Commit message: Added 2 dof champ urdf, control and launch  files.  Changes to be committed: 	new file:   champ_description/launch/champ2D_world.launch 	new file:   champ_description/urdf/champ2D_bhand.xacro 	modified:   champ_description/urdf/wam/defs/components.urdf.xacro 	new file:   champ_description/urdf/wam/wam2_bhand.urdf.xacro 	new file:   champ_description/urdf/wam/wam2_bhand.xacro 	new file:   wam_control/launch/wam2d_bhand_effort_control.launch 	new file:   wam_control/launch/wam2d_bhand_position_control.launch

File: champ_description/urdf/wam/defs/components.urdf.xacro (robot description, xacro)
@@ -516,3 +516,274 @@
     </link>
   </xacro:macro>
+  <xacro:macro name="wam_2dof" params="prefix parent_link xyz rpy">
+    <joint name="${prefix}/wam_fixed_joint" type="fixed">
+      <parent link="${parent_link}"/>
+      <child link="${prefix}/base_link"/>
+      <origin xyz="${xyz}" rpy="${rpy}"/>
+    </joint>
+    <link name = "${prefix}/base_link">
+      <inertial>
+        <origin xyz="0 0 0" />
+        <mass value="1" />
+        <inertia
+          ixx="0.1" ixy="0"   ixz="0"
+                  iyy="0.1"   iyz="0"
+                            izz="0.1" />
+      </inertial>
+      <visual>
+        <material name="WAMGrey">
+          <color rgba="0.7 0.7 0.7 0.0"/>
+        </material>
+        <geometry>
+          <mesh filename="${models_path}/sw_meshes/base_link_fine.stl"/>
+        </geometry>
+      </visual>
+      <collision>
+        <geometry>
+          <mesh filename="${models_path}/sw_meshes/base_link_convex.dae"/>
+        </geometry>
+      </collision>
+    </link>
+     <joint name="${prefix}/base_yaw_joint" type="revolute">
+      <parent link="${prefix}/base_link"/>
+      <child link="${prefix}/shoulder_yaw_link"/>
+      <origin xyz="0 0 0.346" rpy="0 0 0"/>
+      <axis xyz="0 0 1"/>
+      <limit effort="60" lower="-2.6" upper="2.6" velocity="2.0"/>
+      <dynamics damping="${1.8*b}" friction="0"/>
+    </joint>
+    <gazebo reference="${prefix}/base_yaw_joint">
+      <xacro:gz_joint/>
+    </gazebo>
+    <link name="${prefix}/shoulder_yaw_link" >
+      <inertial>
+        <origin xyz="-.00443422 -.00066489 -0.1289039 " />
+        <mass value="5.0" />
+        <inertia
+          ixx=".13488033"  ixy="-0.00012485"   ixz="0.00213041"
+                           iyy=".09046330"    iyz="-.00068555"
+                                              izz=".11328369" />
+      </inertial>
+      <visual>
+        <material name="WAMGrey">
+          <color rgba="0.7 0.7 0.7 1.0"/>
+        </material>
+        <geometry>
+          <mesh filename="${models_path}/sw_meshes/shoulder_link_fine.stl"/>
+        </geometry>
+      </visual>
+      <collision>
+        <geometry>
+          <mesh filename="${models_path}/sw_meshes/shoulder_link_convex_decomposition.dae"/>
+        </geometry>
+      </collision>
+    </link>
+    <joint name="${prefix}/shoulder_pitch_joint" type="revolute">
+      <parent link="${prefix}/shoulder_yaw_link"/>
+      <child link="${prefix}/shoulder_pitch_link"/>
+      <origin xyz="0 0 0" rpy="${-PI/2} 0 0"/>
+      <axis xyz="0 0 1"/>
+      <limit effort="60" lower="-1.985" upper="1.985" velocity="2.0"/>
+      <dynamics damping="${0.5*b}" friction="0"/>
+    </joint>
+    <gazebo reference="${prefix}/shoulder_pitch_joint">
+      <xacro:gz_joint/>
+    </gazebo>
+    <link name="${prefix}/shoulder_pitch_link" >
+      <visual>
+        <material name="WAMGrey">
+          <color rgba="0.7 0.7 0.7 1.0"/>
+        </material>
+        <geometry>
+          <mesh filename="${models_path}/sw_meshes/shoulder_pitch_link_fine.stl"/>
+        </geometry>
+      </visual>
+      <inertial>
+        <origin xyz="-.00236981 -.01542114 .03105614 " />
+        <mass value="3.87493756" />
+        <inertia
+          ixx="0.02140958"  ixy="-0.00002461"  ixz="0.00027172"
+                            iyy="0.015589060"  iyz="0.0018192"
+                                               izz="0.01377875" />
+      </inertial>
+      <collision>
+        <geometry>
+          <mesh filename="${models_path}/sw_meshes/shoulder_pitch_link_convex.dae"/>
+        </geometry>
+      </collision>
+    </link>
+    <joint name="${prefix}/shoulder_yaw_joint" type="fixed">
+      <parent link="${prefix}/shoulder_pitch_link"/>
+      <child link="${prefix}/upper_arm_link"/>
+      <origin xyz="0 0 0" rpy="${PI/2} 0 0"/>
+    </joint>
+    <gazebo reference="${prefix}/shoulder_yaw_joint">
+      <xacro:gz_joint/>
+    </gazebo>
+    <link name="${prefix}/upper_arm_link" >
+      <inertial>
+        <origin xyz="0.00683258580000000 0.000033090000000 0.392492300000000" />
+        <mass value="2.20228141" />
+        <inertia
+          ixx=".05911077"  ixy="-0.00000738"  ixz="-0.00249612"
+                           iyy="0.05927043"   iyz="0.00001767"
+                                              izz="0.0032455" />
+      </inertial>
+      <visual>
+        <material name="WAMGrey">
+          <color rgba="0.7 0.7 0.7 1.0"/>
+        </material>
+        <geometry>
+          <mesh filename="${models_path}/sw_meshes/upper_arm_link_fine.stl"/>
+        </geometry>
+      </visual>
+      <collision>
+        <geometry>
+          <mesh filename="${models_path}/sw_meshes/upper_arm_link_convex_decomposition.dae"/>
+        </geometry>
+      </collision>
+    </link>
+    <joint name="${prefix}/elbow_pitch_joint" type="fixed">
+      <parent link="${prefix}/upper_arm_link"/>
+      <child link="${prefix}/forearm_link"/>
+      <origin xyz="0.045 0 0.55" rpy="${-PI/2} 0 0"/>
+    </joint>
+    <gazebo reference="${prefix}/elbow_pitch_joint">
+      <xacro:gz_joint/>
+    </gazebo>
+    <link name="${prefix}/forearm_link" >
+      <inertial>
+        <mass value="0.50016804" />
+        <origin xyz="-0.04001488 -.14271662 -.00022942 " rpy="0 0 0" />
+        <inertia
+          ixx="0.01491672" ixy="0.001506040000000" ixz="0.000017410000000"
+                           iyy="0.002944630000000" iyz="0.000021090000000"
+                                                   izz="0.014829880000000" />
+      </inertial>
+      <visual>
+        <material name="WAMGrey">
+          <color rgba="0.7 0.7 0.7 1.0"/>
+        </material>
+        <geometry>
+          <mesh filename="${models_path}/sw_meshes/elbow_link_fine.stl"/>
+        </geometry>
+      </visual>
+      <collision>
+        <geometry>
+          <mesh filename="${models_path}/sw_meshes/elbow_link_convex.dae"/>
+        </geometry>
+      </collision>
+      <visual>
+        <material name="WAMGrey">
+          <color rgba="0.7 0.7 0.7 1.0"/>
+        </material>
+        <origin xyz="-0.045 -0.0730 0" rpy="${PI/2} 0 0" />
+        <geometry>
+          <mesh filename="${models_path}/sw_meshes/forearm_link_fine.stl"/>
+        </geometry>
+      </visual>
+      <collision>
+        <origin xyz="-0.045 -0.0730 0" rpy="${PI/2} 0 0" />
+        <geometry>
+          <mesh filename="${models_path}/sw_meshes/forearm_link_convex_decomposition.dae"/>
+        </geometry>
+      </collision>
+    </link>
+    <joint name="${prefix}/wrist_yaw_joint" type="fixed">
+      <parent link="${prefix}/forearm_link"/>
+      <child link="${prefix}/wrist_yaw_link"/>
+      <origin xyz="-0.045 -0.3 0" rpy="${PI/2} 0 0"/>
+    </joint>
+    <gazebo reference="${prefix}/wrist_yaw_joint">
+      <xacro:gz_joint/>
+    </gazebo>
+    <link name="${prefix}/wrist_yaw_link" >
+      <inertial>
+        <origin xyz="0.00008921 0.00435824 -0.00511217 " />
+        <mass value="1.05376019" />
+        <inertia  ixx="0.00005029" ixy="0.00000020"  ixz="0.00007582"
+          iyy="0.00007582"  iyz="-0.00000359"
+          izz="0.00006270" />
+      </inertial>
+      <visual>
+        <material name="WAMGrey">
+          <color rgba="0.7 0.7 0.7 1.0"/>
+        </material>
+        <origin xyz="0 0 0" rpy="0 0 0" />
+        <geometry>
+          <mesh filename="${models_path}/sw_meshes/wrist_yaw_link_fine.stl"/>
+        </geometry>
+      </visual>
+      <collision>
+        <origin xyz="0 0 0" rpy="0 0 0" />
+        <geometry>
+          <mesh filename="${models_path}/sw_meshes/wrist_yaw_link_convex_decomposition.dae"/>
+        </geometry>
+      </collision>
+    </link>
+    <joint name="${prefix}/wrist_pitch_joint" type="fixed">
+      <parent link="${prefix}/wrist_yaw_link"/>
+      <child link="${prefix}/wrist_pitch_link"/>
+      <origin xyz="0 0 0" rpy="${-PI/2} 0 0"/>
+    </joint>
+    <gazebo reference="${prefix}/wrist_pitch_joint">
+      <xacro:gz_joint/>
+    </gazebo>
+    <link name="${prefix}/wrist_pitch_link" >
+      <inertial>
+        <origin xyz="-0.00012262 -0.02468336 -0.01703194 " rpy="0 0 0" />
+        <mass value="0.51797364" />
+        <inertia
+          ixx="0.00055516"  ixy="0.00000061"  ixz="-0.00000074"
+          iyy="0.00024367"  iyz="-0.00004590"
+          izz="0.00045358" />
+      </inertial>
+      <visual>
+        <material name="WAMGrey">
+          <color rgba="0.7 0.7 0.7 1.0"/>
+        </material>
+        <geometry>
+          <mesh filename="${models_path}/sw_meshes/wrist_pitch_link_fine.stl"/>
+        </geometry>
+      </visual>
+      <collision>
+        <geometry>
+          <mesh filename="${models_path}/sw_meshes/wrist_pitch_link_convex_decomposition.dae"/>
+        </geometry>
+      </collision>
+    </link>
+  <!-- Palm without force-torque sensor -->
+    <joint name="${prefix}/palm_yaw_joint" type="fixed">
+      <parent link="${prefix}/wrist_pitch_link"/>
+      <child link="${prefix}/wrist_palm_link"/>
+      <origin xyz="0 0 0" rpy="${PI/2} 0 0"/>
+    </joint>
+    <gazebo reference="${prefix}/palm_yaw_joint">
+      <xacro:gz_joint/>
+    </gazebo>
+    <link name="${prefix}/wrist_palm_link" >
+      <inertial>
+        <origin xyz="0.0 0.0 0.055" rpy="0 0 0" />
+        <mass value="0.08286134" />
+        <inertia  ixx="0.00010859" ixy="0.00000000"  ixz="-0.00000000"
+          iyy="0.00020683"  iyz="-0.0000000"
+          izz="0.00010851" />
+      </inertial>
+      <visual>
+        <material name="WAMGrey">
+          <color rgba="0.7 0.7 0.7 1.0"/>
+        </material>
+        <origin xyz="0 0 0" rpy="0 0 0" />
+        <geometry>
+          <mesh filename="${models_path}/sw_meshes/wrist_palm_link_fine.stl"/>
+        </geometry>
+      </visual>
+      <collision>
+        <origin xyz="0 0 0" rpy="0 0 0" />
+        <geometry>
+          <mesh filename="${models_path}/sw_meshes/wrist_palm_link_convex.dae"/>
+        </geometry>
+      </collision>
+    </link>
+  </xacro:macro>
 </robot>
