Commit message: - Fixed exploding joints problem for champ_bhand.launch - Fixed independent launch (Launching arm without powerbot base) of WAM arm and related controller  Issues:         - WAM collision meshes have holes.         - WAM joint PID parameters still untuned.         - Still need to fix inertias and surface friction for base wheels (currently disabled).

File: champ_description/urdf/champ_bhand.xacro (robot description, xacro)
@@ -30,5 +30,5 @@
 <joint name="world_fixed_joint" type="fixed">
 <!--NB!: origin of base_center is in the center of the chassis, therefore we need to offset the base along z-axis to avoing collisions with the floor-->
-<origin xyz="0 0 0" rpy="0 0 0.2"/>
+<origin xyz="0 0 0.2" rpy="0 0 0"/>
 <parent link="world"/>
 <child link="base_center"/>

File: champ_description/urdf/wam/wam7_bball.urdf.xacro (robot description, xacro)
@@ -96,3 +96,8 @@
     </actuator>
   </transmission>
+<gazebo>
+  <plugin name="gazebo_ros_control" filename="libgazebo_ros_control.so">
+    <robotNamespace>/wam_powerbot</robotNamespace>
+  </plugin>
+</gazebo>
 </robot>

File: champ_description/urdf/wam/wam7_bhand.urdf.xacro (robot description, xacro)
@@ -191,3 +191,8 @@
     </actuator>
   </transmission>
+<gazebo>
+  <plugin name="gazebo_ros_control" filename="libgazebo_ros_control.so">
+    <robotNamespace>/wam_powerbot</robotNamespace>
+  </plugin>
+</gazebo>
 </robot>
